File: Digitronevé hod/LV part/Digitronove hodiny LV-backups/Digitronove hodiny LV-2025-12-21_193653/Digitronove hodiny LV.kicad_sch (KiCad schematic)
At the start: 92 parts, among them J1 DD4012SB_3V3, J10 Output, J11 Output, J12 Output, J13 -, J14 9V to 170V, J15 Output, J16 Output, J17 Output, J18 Output, J19 Output, J2 +, J20 Output, J21 Output, J22 Output, J23 Output, J24 Output, J25 Output, J26 Output, J27 Output, J28 Output, J29 Output, J3 Output, J30 Output, J31 Output, J32 Output, J33 Output, J34 RCWL-0516, J35 Output, J36 Output, J37 Output, J38 Output, J39 Output, J4 Output, J40 Output, J41 Output, J42 Output, J5 Output, J6 Output, J7 Output, J8 Output, J9 Output, SW1 RESET, SW2 SWITCH, SW3 +1, SW4 START/STOP, U1 74HC595, U2 74HC595, U3 ESP32-WROOM-32, U4 74HC595, U5 74HC595, U6 74HC595, U7 74HC595

Commit message: schéma LV desky update
Parts:
- removed J24: Output, Connector_PinHeader_2.00mm:PinHeader_1x01_P2.00mm_Horizontal, symbol Connector_Generic:Conn_01x01
- removed R11, R2, R21: 470, Resistor_SMD:R_1206_3216Metric_Pad1.30x1.75mm_HandSolder, symbol Device:R
- added J34: Output, symbol Connector_Generic:Conn_01x01
- added R1, R3, R40: 470, symbol Device:R
- J10, J11, J12, J15, J16, J17, J18, J19, J20, J21, J22, J25, J26, J27, J28, J29, J3, J30, J31, J32, J33, J35, J36, J37, J38, J39, J4, J40, J41, J42, J5, J6, J7, J8, J9: footprint Connector_PinHeader_2.00mm:PinHeader_1x01_P2.00mm_Horizontal -> (none)
- J43: renamed from J23; footprint Connector_PinHeader_2.00mm:PinHeader_1x01_P2.00mm_Horizontal -> (none)
- R10, R12, R13, R14, R15, R16, R17, R18, R19, R20, R22, R23, R24, R25, R26, R27, R28, R29, R30, R31, R32, R33, R34, R35, R36, R37, R38, R39, R4, R5, R6, R7, R8, R9: footprint Resistor_SMD:R_1206_3216Metric_Pad1.30x1.75mm_HandSolder -> (none)
- R11: renamed from R1; footprint Resistor_SMD:R_1206_3216Metric_Pad1.30x1.75mm_HandSolder -> (none)
- R2: renamed from R3; footprint Resistor_SMD:R_1206_3216Metric_Pad1.30x1.75mm_HandSolder -> (none)
- U1, U2, U4, U5, U6, U7: footprint LOGIC-74HC595N_DIP16_:DIP16-2.54-20.32X5.84MM -> (none)
- renumbered J34 to J24, SW4 to SW2, SW2 to SW4
Connections:
- net at J6.1 (Pin_1): now also R4.1; no longer R5.1
- net at R31.1: now also J34.1 (Pin_1); no longer J33.1 (Pin_1)
- net at R18.1: now also J20.1 (Pin_1); no longer J19.1 (Pin_1)
- net at U4.3 (QD): now also R17.2; no longer R18.2
- net at R7.1: now also J9.1 (Pin_1); no longer J8.1 (Pin_1)
- net at R7.2: now also U2.3 (QD); no longer U2.4 (QE)
- net at J22.1 (Pin_1): now also R20.1
- net at U4.15 (QA): now also R20.2
- net at R29.1: now also J32.1 (Pin_1); no longer J31.1 (Pin_1)
- net at R26.1: now also J29.1 (Pin_1); no longer J28.1 (Pin_1)
- net at J18.1 (Pin_1): now also R16.1; no longer R17.1
- net at U4.4 (QE): now also R16.2; no longer R17.2
- net at R27.1: now also J30.1 (Pin_1); no longer J29.1 (Pin_1)
- net at J17.1 (Pin_1): now also R15.1; no longer R16.1
- net at U4.5 (QF): now also R15.2; no longer R16.2
- net at J26.1 (Pin_1): now also R23.1; no longer R24.1
- net at R22.1: now also J25.1 (Pin_1)
- net at R14.1: now also J16.1 (Pin_1); no longer J15.1 (Pin_1)
- net at J5.1 (Pin_1): now also R3.1; no longer R4.1
- net at J11.1 (Pin_1): now also R9.1; no longer R10.1
- net at U3.33 (IO21): now also R40.2; no longer R13.2
- net at R6.1: now also J8.1 (Pin_1); no longer J7.1 (Pin_1)
- net at R6.2: now also U2.4 (QE); no longer U2.5 (QF)
- net at J10.1 (Pin_1): now also R8.1; no longer R9.1
- net at U2.2 (QC): now also R8.2; no longer R9.2
- net at R14.2: now also U4.6 (QG); no longer U4.7 (QH)
- net at U4.1 (QB): now also R19.2; no longer R20.2
- net at U4.2 (QC): now also R18.2; no longer R19.2
- net at R13.1: now also J15.1 (Pin_1); no longer J43.1 (Pin_1)
- net at R30.1: now also J33.1 (Pin_1); no longer J32.1 (Pin_1)
- net at R19.1: now also J21.1 (Pin_1); no longer J20.1 (Pin_1)
- net at J3.1 (Pin_1): now also R1.1
- net at U1.1 (QB): now also R1.2
- net at U2.7 (QH): now also R3.2; no longer R4.2
- net at R25.1: now also J28.1 (Pin_1); no longer J27.1 (Pin_1)
- net at R28.1: now also J31.1 (Pin_1); no longer J30.1 (Pin_1)
- net at J12.1 (Pin_1): now also R10.1
- net at U2.15 (QA): now also R10.2
- net at U2.1 (QB): now also R9.2; no longer R10.2
- net at U2.6 (QG): now also R4.2; no longer R5.2
- new net: J19.1 (Pin_1), R17.1
- new net: R13.2, U4.7 (QH)
- new net: J27.1 (Pin_1), R24.1
- new net: J7.1 (Pin_1), R5.1
- new net: J43.1 (Pin_1), R40.1
- new net: R5.2, U2.5 (QF)
