File: Digitronevé hod/HV part/Digitronove hodiny LV.kicad_sch (KiCad schematic)
At the start: 25 parts, among them J1 StepDown 5V-3,3V, J2 USB C s 5.1k rezitory, J3 Conn_01x05, Q1 MPSA42, Q13 MPSA42, SW1 SW_Push, SW2 SW_Push, SW3 SW_Push, SW4 SW_Push, SW5 SW_Push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

Commit message: HV part schematic 01
Parts:
- removed C1: 100 uF, symbol Device:C
- removed C2, C3: 47 uF, symbol Device:C
- removed C4: 4.7 uF, symbol Device:C
- removed F1: Fuse, symbol Device:Fuse
- removed J1: StepDown 5V-3,3V, symbol Connector_Generic:Conn_01x03
- removed J2: USB C s 5.1k rezitory, symbol Connector_Generic:Conn_01x02
- removed J3: Conn_01x05, symbol Connector_Generic:Conn_01x05
- removed Q1, Q13: MPSA42, Package_TO_SOT_THT:TO-92_Inline, symbol Transistor_BJT:MPSA42
- removed R13: 100k, symbol Device:R
- removed R14: 470, symbol Device:R
- removed R4: R_Trim, symbol Device:R_Trim
- removed SW1, SW2, SW3, SW4, SW5: SW_Push, symbol Switch:SW_Push
- removed U2: ESP32-WROOM-32, RF_Module:ESP32-WROOM-32, symbol RF_Module:ESP32-WROOM-32
- removed U3, U4: 74HC595, symbol 74xx:74HC595
- added 170V: Conn_01x02, symbol Connector_Generic:Conn_01x02
- added J1: 3V3, symbol Connector_Generic:Conn_01x01
- added J2: RCLK, symbol Connector_Generic:Conn_01x01
- added J3: SER, symbol Connector_Generic:Conn_01x01
- added J4: SRCLK, symbol Connector_Generic:Conn_01x01
- added J5: 5V, symbol Connector_Generic:Conn_01x01
- added J6, J7: GND, symbol Connector_Generic:Conn_01x01
- added R4: 10K, symbol Device:R
- added U10, U7, U8, U9: IN-14, symbol custom:IN-14
- added U2: 74HC595, symbol 74xx:74HC595
- added U3, U4, U5, U6: ~, symbol custom:K155ID1
- R1: value 470 -> 10K
- R2: value 100k -> 10K
- R3: value 10 k -> 10K
Connections:
- net GND: now also U1.8 (GND), 170V.GND (Pin_2), J6.1 (Pin_1), J7.1 (Pin_1), U2.8 (GND), U3. (Q9), U4. (Q9), U5. (Q9), U6. (Q9); no longer R2.2
- net at R2.1: now also U9. (C_comma); no longer R1.2
- net at R3.1: now also U8. (C_comma)
- net at U1.15 (QA): now also U6. (Q9); no longer R1.1
- net at R3.2: now also R1.2, R2.2, 170V.170V (Pin_1), R4.2
- net at U1.1 (QB): now also U6. (Q9)
- net at U1.11 (SRCLK): now also J4.1 (Pin_1), U2.11 (SRCLK)
- net at U1.12 (RCLK): now also J2.1 (Pin_1), U2.12 (RCLK)
- net at U1.14 (SER): now also J3.1 (Pin_1)
- net at U1.16 (VCC): now also J1.1 (Pin_1), U2.16 (VCC)
- net at U1.2 (QC): now also U6. (Q9)
- net at U1.3 (QD): now also U6. (Q9)
- net at U1.4 (QE): now also U5. (Q9)
- net at U1.5 (QF): now also U5. (Q9)
- net at U1.6 (QG): now also U5. (Q9)
- net at U1.7 (QH): now also U5. (Q9)
- net at U1.9 (QH'): now also U2.14 (SER)
- new net: J5.1 (Pin_1), U3. (Q9), U4. (Q9), U5. (Q9), U6. (Q9)
- new net: U3. (Q9), U7. (C_comma) (x10)
- new net: U2.4 (QE), U3. (Q9)
- new net: U2.5 (QF), U3. (Q9)
- new net: U2.6 (QG), U3. (Q9)
- new net: U2.7 (QH), U3. (Q9)
- new net: R4.1, U7. (C_comma)
- new net: U4. (Q9), U8. (C_comma) (x10)
- new net: U5. (Q9), U9. (C_comma) (x10)
- new net: U2.1 (QB), U4. (Q9)
- new net: U2.15 (QA), U4. (Q9)
- new net: U2.2 (QC), U4. (Q9)
- new net: U2.3 (QD), U4. (Q9)
- new net: R1.1, U10. (C_comma)
- new net: U10. (C_comma), U6. (Q9) (x10)
- no-connect marks 3 -> 10

Commit message: HV scheme update
Parts:
- added J8: ESP32, symbol Connector_Generic:Conn_01x01
- added NE1: Lamp_Neon, symbol Device:Lamp_Neon
- added Q1: MPSA42, Package_TO_SOT_THT:TO-92_Inline, symbol Transistor_BJT:MPSA42
- added R5: 10K, symbol Device:R
- added R7: 180K, symbol Device:R
Connections:
- net GND: now also Q1.3 (C), R5.2
- net at U7. (C_comma): now also R4.1; no longer U3. (Q9)
- net at U8. (C_comma): now also R3.1
- net at U9. (C_comma): now also R2.1
- net at 170V.170V (Pin_1), R1.2, R2.2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: now also R7.2
- net at U10. (C_comma): no longer U6. (Q9)
- new net: J8.1 (Pin_1), Q1.2 (B), R5.1
- new net: J5.1 (Pin_1), U3. (Q9), U4. (Q9), U5. (Q9), U6. (Q9)
- new net: U3. (Q9), U7. (C_comma) (x10)
- new net: U4. (Q9), U8. (C_comma) (x10)
- new net: NE1.1, R7.1
- new net: NE1.2, Q1.1 (E)
- new net: U5. (Q9), U9. (C_comma) (x10)
- new net: U10. (C_comma), U6. (Q9) (x10)
- now unconnected: U10. (C_comma), U10. (C_comma), U10. (C_comma), U10. (C_comma), U10. (C_comma), U10. (C_comma), U10. (C_comma), U10. (C_comma), U10. (C_comma)
Other:
- moved on the sheet: 170V

Commit message: LV update
Parts:
- U1, U2: footprint (none) -> LOGIC-74HC595N_DIP16_:74HC595N
Connections:
- net at U7. (C_comma): now also R4.1; no longer U3. (Q9)
- net at U8. (C_comma): now also R3.1
- net at U9. (C_comma): now also R2.1
- net at U10. (C_comma): no longer U6. (Q9)
- new net: J5.1 (Pin_1), U3. (Q9), U4. (Q9), U5. (Q9), U6. (Q9)
- new net: U3. (Q9), U7. (C_comma) (x10)
- new net: U4. (Q9), U8. (C_comma) (x10)
- new net: U5. (Q9), U9. (C_comma) (x10)
- new net: U10. (C_comma), U6. (Q9) (x10)
- now unconnected: U10. (C_comma), U10. (C_comma), U10. (C_comma), U10. (C_comma), U10. (C_comma), U10. (C_comma), U10. (C_comma), U10. (C_comma), U10. (C_comma)
Changed lines of the file:
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@@
 			)
 		)
-		(property "Footprint" ""
+		(property "Footprint" "LOGIC-74HC595N_DIP16_:74HC595N"
 			(at 110.49 49.53 0)
 			(effects
@@
 			)
 		)
-		(property "Footprint" ""
+		(property "Footprint" "LOGIC-74HC595N_DIP16_:74HC595N"
 			(at 58.42 49.53 0)
 			(effects

Commit message: Redesign LV
Parts:
- added C1: C, symbol Device:C
- added C2, C3, C4, C5: C_Small, symbol Device:C_Small
- 170V: footprint (none) -> Connector_PinHeader_1.00mm:PinHeader_2x01_P1.00mm_Vertical
- J1, J2, J3, J4, J5, J6, J7, J8: footprint (none) -> Connector_PinHeader_1.00mm:PinHeader_1x01_P1.00mm_Vertical
- R1, R2, R3, R4, R5, R7: footprint (none) -> Resistor_THT:R_Axial_DIN0207_L6.3mm_D2.5mm_P10.16mm_Horizontal
Connections:
- net GND: now also C2.2, C3.2, C4.2, C5.2
- net at U7. (C_comma): now also R4.1; no longer U3. (Q9)
- net at U8. (C_comma): now also R3.1
- net at R1.2, R2.2, R3.2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: now also C1.1; no longer 170V.170V (Pin_1)
- net at U9. (C_comma): now also R2.1
- net at U10. (C_comma): no longer U6. (Q9)
- new net: C2.1, C3.1, C4.1, C5.1, J5.1 (Pin_1), U3. (Q9), U4. (Q9), U5. (Q9), U6. (Q9)
- new net: 170V.170V (Pin_1), C1.2
- new net: U3. (Q9), U7. (C_comma) (x10)
- new net: U4. (Q9), U8. (C_comma) (x10)
- new net: U5. (Q9), U9. (C_comma) (x10)
- new net: U10. (C_comma), U6. (Q9) (x10)
- now unconnected: U10. (C_comma), U10. (C_comma), U10. (C_comma), U10. (C_comma), U10. (C_comma), U10. (C_comma), U10. (C_comma), U10. (C_comma), U10. (C_comma)
Other:
- moved on the sheet: 170V

Commit message: Před kontrolou
Parts:
- added C1: 470 µF, Capacitor_THT:CP_Radial_D5.0mm_P2.50mm, symbol Device:C_Small
- added C7, C8: 100 nF, Capacitor_SMD:C_1206_3216Metric_Pad1.33x1.80mm_HandSolder, symbol Device:C_Small
- added NE1: Lamp_Neon, Capacitor_THT:CP_Radial_D5.0mm_P2.50mm, symbol Device:Lamp_Neon
- added R6: 180K, Resistor_THT:R_Axial_DIN0207_L6.3mm_D2.5mm_P10.16mm_Horizontal, symbol Device:R
- 170V1: renamed from 170V; footprint Connector_PinHeader_1.00mm:PinHeader_2x01_P1.00mm_Vertical -> Connector_PinHeader_2.00mm:PinHeader_1x02_P2.00mm_Vertical
- C2, C3, C4, C5: value C_Small -> 100 nF; footprint (none) -> Capacitor_SMD:C_1206_3216Metric_Pad1.33x1.80mm_HandSolder
- C6: renamed from C1; value C -> 4.7 µF; footprint (none) -> Capacitor_THT:CP_Radial_D10.0mm_P5.00mm
- J1, J8: footprint Connector_PinHeader_1.00mm:PinHeader_1x01_P1.00mm_Vertical -> Connector_PinHeader_2.00mm:PinHeader_1x01_P2.00mm_Vertical
- J2: renamed from J6; footprint Connector_PinHeader_1.00mm:PinHeader_1x01_P1.00mm_Vertical -> Connector_PinHeader_2.00mm:PinHeader_1x01_P2.00mm_Vertical
- J3: renamed from J7; footprint Connector_PinHeader_1.00mm:PinHeader_1x01_P1.00mm_Vertical -> Connector_PinHeader_2.00mm:PinHeader_1x01_P2.00mm_Vertical
- J4: renamed from J2; footprint Connector_PinHeader_1.00mm:PinHeader_1x01_P1.00mm_Vertical -> Connector_PinHeader_2.00mm:PinHeader_1x01_P2.00mm_Vertical
- J5: renamed from J4; footprint Connector_PinHeader_1.00mm:PinHeader_1x01_P1.00mm_Vertical -> Connector_PinHeader_2.00mm:PinHeader_1x01_P2.00mm_Vertical
- J6: renamed from J3; footprint Connector_PinHeader_1.00mm:PinHeader_1x01_P1.00mm_Vertical -> Connector_PinHeader_2.00mm:PinHeader_1x01_P2.00mm_Vertical
- J7: renamed from J5; footprint Connector_PinHeader_1.00mm:PinHeader_1x01_P1.00mm_Vertical -> Connector_PinHeader_2.00mm:PinHeader_1x01_P2.00mm_Vertical
- NE2: renamed from NE1; footprint (none) -> Capacitor_THT:CP_Radial_D5.0mm_P2.50mm
- U10, U7, U8, U9: value IN-14 -> ~; footprint (none) -> LOGIC-74HC595N_DIP16_:Tesla_ZM1082
- U3, U4, U5, U6: footprint (none) -> LOGIC-74HC595N_DIP16_:74141
- renumbered R5 to R1, R4 to R2, R2 to R4, R1 to R5, U2 to U1, U1 to U2
Connections:
- net GND: now also 170V1.2 (GND), U3.12 (GND), U4.12 (GND), U5.12 (GND), U6.12 (GND), C7.1, C8.1; no longer 170V1.GND (Pin_2), U3. (Q9), U4. (Q9), U5. (Q9), U6. (Q9)
- net at C2.1, C3.1, C4.1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: now also U3.5 (VCC), U4.5 (VCC), U5.5 (VCC), U6.5 (VCC); no longer U3. (Q9), U4. (Q9), U5. (Q9), U6. (Q9)
- net at C6.1, R2.2, R3.2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: now also R6.2
- net at C6.2: now also 170V1.1 (170V); no longer 170V1.170V (Pin_1)
- net at U1.4 (QE): now also U3.3 (A); no longer U3. (Q9)
- net at U1.5 (QF): now also U3.6 (B); no longer U3. (Q9)
- net at U1.6 (QG): now also U3.7 (C); no longer U3. (Q9)
- net at U1.7 (QH): now also U3.4 (D); no longer U3. (Q9)
- net at R2.1: now also U7.13 (a); no longer U7. (C_comma)
- net at R3.1: now also U8.13 (a); no longer U8. (C_comma)
- net at NE2.2, Q1.1 (E): now also NE1.2
- net at R4.1: now also U9.13 (a); no longer U9. (C_comma)
- net at U2.1 (QB): now also U6.6 (B); no longer U6. (Q9)
- net at U2.15 (QA): now also U6.3 (A); no longer U6. (Q9)
- net at U1.16 (VCC), U2.16 (VCC): now also C1.2, C7.2, C8.2; no longer J1.1 (Pin_1)
- net at U2.2 (QC): now also U6.7 (C); no longer U6. (Q9)
- net at U2.3 (QD): now also U6.4 (D); no longer U6. (Q9)
- net at U2.4 (QE): now also U5.3 (A); no longer U5. (Q9)
- net at U2.5 (QF): now also U5.6 (B); no longer U5. (Q9)
- net at U2.6 (QG): now also U5.7 (C); no longer U5. (Q9)
- net at U2.7 (QH): now also U5.4 (D); no longer U5. (Q9)
- net at U1.1 (QB): now also U4.6 (B); no longer U4. (Q9)
- net at U1.15 (QA): now also U4.3 (A); no longer U4. (Q9)
- net at U1.2 (QC): now also U4.7 (C); no longer U4. (Q9)
- net at U1.3 (QD): now also U4.4 (D); no longer U4. (Q9)
- net at R5.1: now also U10.13 (a); no longer U10. (C_comma)
- new net: U10.1 (k1), U6.1 (Q8)
- new net: U10.2 (k2), U6.10 (Q7)
- new net: U10.3 (k3), U6.11 (Q6)
- new net: U10.6 (k5), U6.13 (Q4)
- new net: U10.5 (k4), U6.14 (Q5)
- new net: U10.9 (k8), U6.15 (Q1)
- new net: U10.11 (k9), U6.16 (Q0)
- new net: U10.12 (k0), U6.2 (Q9)
- new net: U10.8 (k7), U6.8 (Q2)
- new net: U10.7 (k6), U6.9 (Q3)
- new net: U5.1 (Q8), U9.1 (k1)
- new net: U5.10 (Q7), U9.2 (k2)
- new net: U5.11 (Q6), U9.3 (k3)
- new net: U5.13 (Q4), U9.6 (k5)
- new net: U5.14 (Q5), U9.5 (k4)
- new net: U5.15 (Q1), U9.9 (k8)
- new net: U5.16 (Q0), U9.11 (k9)
- new net: U5.2 (Q9), U9.12 (k0)
- new net: U5.8 (Q2), U9.8 (k7)
- new net: U5.9 (Q3), U9.7 (k6)
- new net: NE1.1, R6.1
- new net: U4.1 (Q8), U8.1 (k1)
- new net: U4.16 (Q0), U8.11 (k9)
- new net: U4.2 (Q9), U8.12 (k0)
- new net: U4.10 (Q7), U8.2 (k2)
- new net: U4.11 (Q6), U8.3 (k3)
- new net: U4.14 (Q5), U8.5 (k4)
- new net: U4.13 (Q4), U8.6 (k5)
- new net: U4.9 (Q3), U8.7 (k6)
- new net: U4.8 (Q2), U8.8 (k7)
- new net: U4.15 (Q1), U8.9 (k8)
- new net: C1.1, J1.1 (Pin_1)
- new net: U3.1 (Q8), U7.1 (k1)
- new net: U3.16 (Q0), U7.11 (k9)
- new net: U3.2 (Q9), U7.12 (k0)
- new net: U3.10 (Q7), U7.2 (k2)
- new net: U3.11 (Q6), U7.3 (k3)
- new net: U3.14 (Q5), U7.5 (k4)
- new net: U3.13 (Q4), U7.6 (k5)
- new net: U3.9 (Q3), U7.7 (k6)
- new net: U3.8 (Q2), U7.8 (k7)
- new net: U3.15 (Q1), U7.9 (k8)
- no-connect marks 10 -> 15
Other:
- moved on the sheet: J1, J6, J8
