File: Digitronevé hod/HV part/Digitronove hodiny LV.kicad_sch (KiCad schematic)
At the start: 41 parts, among them J1 3V3, J2 GND, J3 GND, J4 RCLK, J5 SRCLK, J6 SER, J7 5V, J8 ESP32, Q1 MPSA42, U1 74HC595, U2 74HC595

Commit message: pcb uprava
Parts:
- removed 170V1: Conn_01x02, Connector_PinHeader_2.00mm:PinHeader_1x02_P2.00mm_Vertical, symbol Connector_Generic:Conn_01x02
- removed J1: 3V3, Connector_PinHeader_2.00mm:PinHeader_1x01_P2.00mm_Vertical, symbol Connector_Generic:Conn_01x01
- removed J2, J3: GND, Connector_PinHeader_2.00mm:PinHeader_1x01_P2.00mm_Vertical, symbol Connector_Generic:Conn_01x01
- removed J4: RCLK, Connector_PinHeader_2.00mm:PinHeader_1x01_P2.00mm_Vertical, symbol Connector_Generic:Conn_01x01
- removed J5: SRCLK, Connector_PinHeader_2.00mm:PinHeader_1x01_P2.00mm_Vertical, symbol Connector_Generic:Conn_01x01
- removed J6: SER, Connector_PinHeader_2.00mm:PinHeader_1x01_P2.00mm_Vertical, symbol Connector_Generic:Conn_01x01
- removed J7: 5V, Connector_PinHeader_2.00mm:PinHeader_1x01_P2.00mm_Vertical, symbol Connector_Generic:Conn_01x01
- removed J8: ESP32, Connector_PinHeader_2.00mm:PinHeader_1x01_P2.00mm_Vertical, symbol Connector_Generic:Conn_01x01
- added C9: 100 uF, Capacitor_THT:CP_Radial_D6.3mm_P2.50mm, symbol Device:C_Small
- added J1: Conn_01x02, Connector_JST:JST_EH_B2B-EH-A_1x02_P2.50mm_Vertical, symbol Connector_Generic:Conn_01x02
- added J2: Conn_01x09, Connector_JST:JST_EH_B9B-EH-A_1x09_P2.50mm_Vertical, symbol Connector_Generic:Conn_01x09
- added R9: 1k, Resistor_THT:R_Axial_DIN0207_L6.3mm_D2.5mm_P10.16mm_Horizontal, symbol Device:R
- C1: value 470uF -> 100 uF; footprint Capacitor_THT:CP_Radial_D5.0mm_P2.50mm -> Capacitor_THT:CP_Radial_D6.3mm_P2.50mm
- NE1, NE2: footprint Capacitor_THT:CP_Radial_D5.0mm_P2.50mm -> Capacitor_THT:C_Rect_L4.0mm_W2.5mm_P2.50mm
- R1: value 10K -> 100K
- R2, R3, R4, R5: value 10K -> 10k
- R6, R7: value 180K -> 180k
- U3, U4, U5, U6: value ~ -> K155id1
Connections:
- net GND: now also C8.2, J1.1 (Pin_1), J2.4 (Pin_4), J2.5 (Pin_5)
- net +3V3: now reaches C1.2, C2.2, C3.2, U1.16 (VCC), U2.16 (VCC)
- net +3V3: now also C1.1, U1.10 (~{SRCLR}), U2.10 (~{SRCLR}), J2.3 (Pin_3)
- net +170V: now reaches C8.1, R2.2, R3.2, R4.2, R5.2, R6.2, R7.2, R8.2
- net +170V: now also NE1.1, NE1.2, NE2.1, NE2.2, Q1.1 (E), R2.1, R3.1, R4.1, R5.1, R6.1, R7.1, U10.13 (a), U7.13 (a), U8.13 (a), U9.13 (a), J1.2 (Pin_2), R9.1, R9.2
- net 8a: now reaches U10.1 (k1), U6.1 (Q8)
- net 7a: now reaches U10.2 (k2), U6.10 (Q7)
- net 6a: now reaches U10.3 (k3), U6.11 (Q6)
- net 4a: now reaches U10.6 (k5), U6.13 (Q4)
- net 5a: now reaches U10.5 (k4), U6.14 (Q5)
- net 1a: now reaches U10.9 (k8), U6.15 (Q1)
- net 0a: now reaches U10.11 (k9), U6.16 (Q0)
- net 9a: now reaches U10.12 (k0), U6.2 (Q9)
- net A1: now reaches U2.15 (QA), U6.3 (A)
- net D1: now reaches U2.3 (QD), U6.4 (D)
- net at C4.1, C5.1, C6.1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: now also C9.2
- net B1: now reaches U2.1 (QB), U6.6 (B)
- net C1: now reaches U2.2 (QC), U6.7 (C)
- net 2a: now reaches U10.8 (k7), U6.8 (Q2)
- net 3a: now reaches U10.7 (k6), U6.9 (Q3)
- net NE1,2: now reaches Q1.2 (B), R1.1
- net NE1,2: now also J2.1 (Pin_1)
- net 8b: now reaches U5.1 (Q8), U9.1 (k1)
- net 7b: now reaches U5.10 (Q7), U9.2 (k2)
- net 6b: now reaches U5.11 (Q6), U9.3 (k3)
- net 4b: now reaches U5.13 (Q4), U9.6 (k5)
- net 5b: now reaches U5.14 (Q5), U9.5 (k4)
- net 1b: now reaches U5.15 (Q1), U9.9 (k8)
- net 0b: now reaches U5.16 (Q0), U9.11 (k9)
- net 9b: now reaches U5.2 (Q9), U9.12 (k0)
- net A2: now reaches U2.4 (QE), U5.3 (A)
- net D2: now reaches U2.7 (QH), U5.4 (D)
- net B2: now reaches U2.5 (QF), U5.6 (B)
- net C2: now reaches U2.6 (QG), U5.7 (C)
- net 2b: now reaches U5.8 (Q2), U9.8 (k7)
- net 3b: now reaches U5.9 (Q3), U9.7 (k6)
- net RLCK: now reaches U1.12 (RCLK), U2.12 (RCLK)
- net RLCK: now also J2.7 (Pin_7)
- net SRLCK: now reaches U1.11 (SRCLK), U2.11 (SRCLK)
- net SRLCK: now also J2.6 (Pin_6)
- net 8c: now reaches U4.1 (Q8), U8.1 (k1)
- net 0c: now reaches U4.16 (Q0), U8.11 (k9)
- net 9c: now reaches U4.2 (Q9), U8.12 (k0)
- net 7c: now reaches U4.10 (Q7), U8.2 (k2)
- net 6c: now reaches U4.11 (Q6), U8.3 (k3)
- net 5c: now reaches U4.14 (Q5), U8.5 (k4)
- net 4c: now reaches U4.13 (Q4), U8.6 (k5)
- net 3c: now reaches U4.9 (Q3), U8.7 (k6)
- net 2c: now reaches U4.8 (Q2), U8.8 (k7)
- net 1c: now reaches U4.15 (Q1), U8.9 (k8)
- net OE: now reaches U2.13 (~{OE})
- net OE: now also U1.13 (~{OE}), J2.8 (Pin_8)
- net SER1: now reaches U2.14 (SER)
- net SER1: now also J2.9 (Pin_9)
- net SER2: now reaches U1.14 (SER), U2.9 (QH')
- net A3: now reaches U1.15 (QA), U4.3 (A)
- net D3: now reaches U1.3 (QD), U4.4 (D)
- net B3: now reaches U1.1 (QB), U4.6 (B)
- net C3: now reaches U1.2 (QC), U4.7 (C)
- net A4: now reaches U1.4 (QE), U3.3 (A)
- net B4: now reaches U1.5 (QF), U3.6 (B)
- net C4: now reaches U1.6 (QG), U3.7 (C)
- net D4: now reaches U1.7 (QH), U3.4 (D)
- net 8d: now reaches U3.1 (Q8), U7.1 (k1)
- net 0d: now reaches U3.16 (Q0), U7.11 (k9)
- net 9d: now reaches U3.2 (Q9), U7.12 (k0)
- net 7d: now reaches U3.10 (Q7), U7.2 (k2)
- net 6d: now reaches U3.11 (Q6), U7.3 (k3)
- net 5d: now reaches U3.14 (Q5), U7.5 (k4)
- net 4d: now reaches U3.13 (Q4), U7.6 (k5)
- net 3d: now reaches U3.9 (Q3), U7.7 (k6)
- net 2d: now reaches U3.8 (Q2), U7.8 (k7)
- net 1d: now reaches U3.15 (Q1), U7.9 (k8)
- new net +5V: C9.1, J2.2 (Pin_2)
- no-connect marks 15 -> 11
Other:
- moved on the sheet: C2, C3, C8, R1, R8

Commit message: release meee
Parts:
- removed R9: 1k, Resistor_THT:R_Axial_DIN0207_L6.3mm_D2.5mm_P10.16mm_Horizontal, symbol Device:R
- R1: value 100K -> 10K
Other:
- title: (none) -> Příloha II.
Changed lines of the file:
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@@
 	(generator_version "9.0")
 	(paper "A4")
+	(title_block
+		(title "Příloha II.")
+		(date "08.04.2026")
+		(rev "Augusta Jan")
+		(comment 1 "Horní PCB")
+	)
 	(junction
 		(at 167.64 172.72)
@@
 	(wire
 		(pts
-			(xy 167.64 187.96) (xy 167.64 184.15)
-		)
-		(stroke
-			(width 0)
-			(type default)
-		)
-	)
-	(wire
-		(pts
 			(xy 130.81 31.75) (xy 130.81 49.53)
 		)
@@
 	(wire
 		(pts
+			(xy 167.64 172.72) (xy 167.64 187.96)
+		)
+		(stroke
+			(width 0)
+			(type default)
+		)
+	)
+	(wire
+		(pts
 			(xy 87.63 102.87) (xy 87.63 144.78)
 		)
@@
 	(wire
 		(pts
-			(xy 167.64 176.53) (xy 167.64 172.72)
-		)
-		(stroke
-			(width 0)
-			(type default)
-		)
-	)
-	(wire
-		(pts
 			(xy 73.66 69.85) (xy 63.5 69.85)
 		)
@@
 		(on_board yes)
 		(dnp no)
-		(fields_autoplaced yes)
 		(property "Reference" "C8"
-			(at 171.45 190.4999 0)
+			(at 171.45 191.77 0)
 			(effects
 				(font
@@
 		)
 		(property "Value" "4.7 µF"
-			(at 171.45 193.0399 0)
+			(at 169.672 193.802 0)
 			(effects
 				(font
@@
 	)
 	(symbol
-		(lib_id "Device:R")
-		(at 167.64 180.34 0)
-		(unit 1)
-		(exclude_from_sim no)
-		(in_bom yes)
-		(on_board yes)
-		(dnp no)
-		(fields_autoplaced yes)
-		(property "Reference" "R9"
-			(at 170.18 179.0699 0)
-			(effects
-				(font
-					(size 1.27 1.27)
-				)
-				(justify left)
-			)
-		)
-		(property "Value" "1k"
-			(at 170.18 181.6099 0)
-			(effects
-				(font
-					(size 1.27 1.27)
-				)
-				(justify left)
-			)
-		)
-		(property "Footprint" "Resistor_THT:R_Axial_DIN0207_L6.3mm_D2.5mm_P10.16mm_Horizontal"
-			(at 165.862 180.34 90)
-			(effects
-				(font
-					(size 1.27 1.27)
-				)
-				(hide yes)
-			)
-		)
-		(property "Datasheet" "~"
-			(at 167.64 180.34 0)
-			(effects
-				(font
-					(size 1.27 1.27)
-				)
-				(hide yes)
-			)
-		)
-		(property "Description" "Resistor"
-			(at 167.64 180.34 0)
-			(effects
-				(font
-					(size 1.27 1.27)
-				)
-				(hide yes)
-			)
-		)
-		(pin "2"
-		)
-		(pin "1"
-		)
-		(instances
-			(project "Digitronove hodiny LV"
-				(path "/760f652f-b82b-45ad-92c5-42c0d0511f5b"
-					(reference "R9")
-					(unit 1)
-				)
-			)
-		)
-	)
-	(symbol
 		(lib_id "power:GND")
 		(at 185.42 153.67 0)
@@
 		(fields_autoplaced yes)
 		(property "Reference" "R1"
-			(at 182.88 151.1301 0)
+			(at 187.96 148.5899 0)
 			(effects
 				(font
 					(size 1.27 1.27)
 				)
-				(justify right)
+				(justify left)
 			)
 		)
-		(property "Value" "100K"
-			(at 182.88 148.5901 0)
+		(property "Value" "10K"
+			(at 187.96 151.1299 0)
 			(effects
 				(font
 					(size 1.27 1.27)
 				)
-				(justify right)
+				(justify left)
 			)
 		)
