File: Digitronevé hod/HV part/Digitronove hodiny LV.kicad_pcb (KiCad board)
At the start: 2 copper layers, 136 x 62 mm, 37 parts, among them J1 3V3, J2 GND, J3 GND, J4 RCLK, J5 SRCLK, J6 SER, J7 5V, J8 ESP32, Q1 MPSA42, U1 74HC595, U2 74HC595

Commit message: PCB finnal
Parts:
- added H1: MountingHole, MountingHole:MountingHole_2.5mm, F.Cu at (86.7, 59.7)
- added H2: MountingHole, MountingHole:MountingHole_2.5mm, F.Cu at (215.7, 59.7)
- added H3: MountingHole, MountingHole:MountingHole_2.5mm, F.Cu at (157.2, 114.7)
- added R8: 1M, Resistor_THT:R_Axial_DIN0207_L6.3mm_D2.5mm_P10.16mm_Horizontal, B.Cu at (215.7, 66.6)
- C1: value 470 µF -> 470uF; moved to B.Cu
- C8: renamed from C6; moved to B.Cu
- R1, R6, R7: moved to B.Cu
- moved C3 1.55 mm to (211.9, 105.2)
- renumbered 170V1 to 170V, C7 to C2, C8 to C3, C2 to C4, C3 to C5, C4 to C6, C5 to C7
Routing:
- net Net-(C8-Pad1): track 253.2 -> 261.6 mm
- net Net-(U1-SER): track 210.7 -> 204.3 mm
- net Net-(U3-Q9): track 33.7 -> 31.6 mm
- net Net-(U1-VCC): track 146.6 -> 147.6 mm, vias 1 -> 0
- net Net-(J4-Pin_1): track 154.0 -> 153.4 mm
- net GND: vias 13 -> 12

Commit message: pcb uprava
Parts:
- removed 170V: Conn_01x02, Connector_PinHeader_2.00mm:PinHeader_1x02_P2.00mm_Vertical
- removed J3: GND, Connector_PinHeader_2.00mm:PinHeader_1x01_P2.00mm_Vertical
- removed J4: RCLK, Connector_PinHeader_2.00mm:PinHeader_1x01_P2.00mm_Vertical
- removed J5: SRCLK, Connector_PinHeader_2.00mm:PinHeader_1x01_P2.00mm_Vertical
- removed J6: SER, Connector_PinHeader_2.00mm:PinHeader_1x01_P2.00mm_Vertical
- removed J7: 5V, Connector_PinHeader_2.00mm:PinHeader_1x01_P2.00mm_Vertical
- removed J8: ESP32, Connector_PinHeader_2.00mm:PinHeader_1x01_P2.00mm_Vertical
- added C9: 100 uF, Capacitor_THT:CP_Radial_D6.3mm_P2.50mm, B.Cu at (91.1, 66.1)
- added R9: 1k, Resistor_THT:R_Axial_DIN0207_L6.3mm_D2.5mm_P10.16mm_Horizontal, B.Cu at (214.2, 86.1)
- C1: value 470uF -> 100 uF; footprint Capacitor_THT:CP_Radial_D5.0mm_P2.50mm -> Capacitor_THT:CP_Radial_D6.3mm_P2.50mm
- C2, C3: moved to B.Cu
- J1: value 3V3 -> Conn_01x02; footprint Connector_PinHeader_2.00mm:PinHeader_1x01_P2.00mm_Vertical -> Connector_JST:JST_EH_B2B-EH-A_1x02_P2.50mm_Vertical
- J2: value GND -> Conn_01x09; footprint Connector_PinHeader_2.00mm:PinHeader_1x01_P2.00mm_Vertical -> Connector_JST:JST_EH_B9B-EH-A_1x09_P2.50mm_Vertical
- NE1: footprint Capacitor_THT:CP_Radial_D5.0mm_P2.50mm -> Capacitor_THT:C_Rect_L4.0mm_W2.5mm_P2.50mm; moved to F.Cu
- NE2: footprint Capacitor_THT:CP_Radial_D5.0mm_P2.50mm -> Capacitor_THT:C_Rect_L4.0mm_W2.5mm_P2.50mm
- R1, R2, R3, R4, R5: value 10K -> 10k
- R6, R7: value 180K -> 180k
- moved J2 79.6 mm to (85.9, 65.7), turned to -90 degrees
- moved C1 70.3 mm to (91.1, 73.2), turned to 0 degrees
- moved J1 64.1 mm to (211.7, 90.5), turned to 0 degrees
- moved C7 33.1 mm to (141.6, 96.3), turned to -90 degrees
- moved R8 20.3 mm to (210.1, 86.1), turned to 90 degrees
- moved C4 18.4 mm to (116.2, 96.3), turned to -90 degrees
- moved C8 13.7 mm to (212.4, 71.9)
- moved C3 11.7 mm to (215.5, 116.4), turned to 180 degrees
- moved C2 10.8 mm to (99.1, 113.1)
- moved C6 8.85 mm to (203.0, 94.8), turned to 0 degrees
- moved C5 8.27 mm to (176.6, 96.3), turned to 0 degrees
Connections:
- net Net-(U1-QA) renamed /A3
- net Net-(U1-QB) renamed /B3
- net Net-(U1-QC) renamed /C3
- net Net-(U1-QD) renamed /D3
- net Net-(U1-QE) renamed /A4
- net Net-(U1-QF) renamed /B4
- net Net-(U1-QG) renamed /C4
- net Net-(U1-QH) renamed /D4
- net Net-(U1-SER) renamed /SER2
- net Net-(U10-k0) renamed /9a
- net Net-(U10-k1) renamed /8a
- net Net-(U10-k2) renamed /7a
- net Net-(U10-k3) renamed /6a
- net Net-(U10-k4) renamed /5a
- net Net-(U10-k5) renamed /4a
- net Net-(U10-k6) renamed /3a
- net Net-(U10-k7) renamed /2a
- net Net-(U10-k8) renamed /1a
- net Net-(U10-k9) renamed /0a
- net Net-(U2-QA) renamed /A1
- net Net-(U2-QB) renamed /B1
- net Net-(U2-QC) renamed /C1
- net Net-(U2-QD) renamed /D1
- net Net-(U2-QE) renamed /A2
- net Net-(U2-QF) renamed /B2
- net Net-(U2-QG) renamed /C2
- net Net-(U2-QH) renamed /D2
- net Net-(U3-Q0) renamed /0d
- net Net-(U3-Q1) renamed /1d
- net Net-(U3-Q2) renamed /2d
- net Net-(U3-Q3) renamed /3d
- net Net-(U3-Q4) renamed /4d
- net Net-(U3-Q5) renamed /5d
- net Net-(U3-Q6) renamed /6d
- net Net-(U3-Q7) renamed /7d
- net Net-(U3-Q8) renamed /8d
- net Net-(U3-Q9) renamed /9d
- net Net-(U4-Q0) renamed /0c
- net Net-(U4-Q1) renamed /1c
- net Net-(U4-Q2) renamed /2c
- net Net-(U4-Q3) renamed /3c
- net Net-(U4-Q4) renamed /4c
- net Net-(U4-Q5) renamed /5c
- net Net-(U4-Q6) renamed /6c
- net Net-(U4-Q7) renamed /7c
- net Net-(U4-Q8) renamed /8c
- net Net-(U4-Q9) renamed /9c
- net Net-(U5-Q0) renamed /0b
- net Net-(U5-Q1) renamed /1b
- net Net-(U5-Q2) renamed /2b
- net Net-(U5-Q3) renamed /3b
- net Net-(U5-Q4) renamed /4b
- net Net-(U5-Q5) renamed /5b
- net Net-(U5-Q6) renamed /6b
- net Net-(U5-Q7) renamed /7b
- net Net-(U5-Q8) renamed /8b
- net Net-(U5-Q9) renamed /9b
- C1 pad 1: Net-(J1-Pin_1) -> /+3V3
- C1 pad 2: Net-(U1-VCC) -> /+3V3
- C2 pad 2: Net-(U1-VCC) -> /+3V3
- C3 pad 2: Net-(U1-VCC) -> /+3V3
- C4 pad 1: Net-(J7-Pin_1) -> /+5V
- C5 pad 1: Net-(J7-Pin_1) -> /+5V
- C6 pad 1: Net-(J7-Pin_1) -> /+5V
- C7 pad 1: Net-(J7-Pin_1) -> /+5V
- C8 pad 1: Net-(C8-Pad1) -> /+170V
- C8 pad 2: Net-(170V1-170V) -> GND
- J1 pad 1: Net-(J1-Pin_1) -> GND
- J2 pad 1: GND -> /NE1,2
- NE1 pad 1: Net-(NE1-Pad1) -> /+170V
- NE1 pad 2: Net-(Q1-E) -> /+170V
- NE2 pad 1: Net-(NE2-Pad1) -> /+170V
- NE2 pad 2: Net-(Q1-E) -> /+170V
- Q1 pad 1: Net-(Q1-E) -> /+170V
- Q1 pad 2: Net-(J8-Pin_1) -> /NE1,2
- R1 pad 1: Net-(J8-Pin_1) -> /NE1,2
- R2 pad 1: Net-(U7-a) -> /+170V
- R2 pad 2: Net-(C8-Pad1) -> /+170V
- R3 pad 1: Net-(U8-a) -> /+170V
- R3 pad 2: Net-(C8-Pad1) -> /+170V
- R4 pad 1: Net-(U9-a) -> /+170V
- R4 pad 2: Net-(C8-Pad1) -> /+170V
- R5 pad 1: Net-(U10-a) -> /+170V
- R5 pad 2: Net-(C8-Pad1) -> /+170V
- R6 pad 1: Net-(NE1-Pad1) -> /+170V
- R6 pad 2: Net-(C8-Pad1) -> /+170V
- R7 pad 1: Net-(NE2-Pad1) -> /+170V
- R7 pad 2: Net-(C8-Pad1) -> /+170V
- R8 pad 2: Net-(C8-Pad1) -> /+170V
- U1 pad 10: unconnected-(U1-~{SRCLR}-Pad10) -> /+3V3
- U1 pad 11: Net-(J5-Pin_1) -> /SRLCK
- U1 pad 12: Net-(J4-Pin_1) -> /RLCK
- U1 pad 13: unconnected-(U1-~{OE}-Pad13) -> /OE
- U1 pad 16: Net-(U1-VCC) -> /+3V3
- U10 pad 13: Net-(U10-a) -> /+170V
- U2 pad 10: unconnected-(U2-~{SRCLR}-Pad10) -> /+3V3
- U2 pad 11: Net-(J5-Pin_1) -> /SRLCK
- U2 pad 12: Net-(J4-Pin_1) -> /RLCK
- U2 pad 13: unconnected-(U2-~{OE}-Pad13) -> /OE
- U2 pad 14: Net-(J6-Pin_1) -> /SER1
- U2 pad 16: Net-(U1-VCC) -> /+3V3
- U3 pad 5: Net-(J7-Pin_1) -> /+5V
- U4 pad 5: Net-(J7-Pin_1) -> /+5V
- U5 pad 5: Net-(J7-Pin_1) -> /+5V
- U6 pad 5: Net-(J7-Pin_1) -> /+5V
- U7 pad 13: Net-(U7-a) -> /+170V
- U8 pad 13: Net-(U8-a) -> /+170V
- U9 pad 13: Net-(U9-a) -> /+170V
Routing:
- net /+170V: track 0.00 -> 312.8 mm
- net /+3V3: track 0.00 -> 266.2 mm, vias 0 -> 5
- net Net-(C8-Pad1): track 261.6 -> 0.00 mm
- net /+5V: track 0.00 -> 231.4 mm, vias 0 -> 7
- net Net-(J7-Pin_1): track 180.9 -> 0.00 mm, vias 3 -> 0
- net /SRLCK: track 0.00 -> 177.6 mm, vias 0 -> 2
- net /RLCK: track 0.00 -> 170.6 mm
- net /OE: track 0.00 -> 168.0 mm, vias 0 -> 4
- net Net-(J5-Pin_1): track 158.0 -> 0.00 mm, vias 2 -> 0
- net Net-(J4-Pin_1): track 153.4 -> 0.00 mm
- net Net-(U1-VCC): track 147.6 -> 0.00 mm
- net /NE1,2: track 0.00 -> 95.6 mm, vias 0 -> 2
- net /SER1: track 0.00 -> 31.3 mm
- net Net-(J6-Pin_1): track 19.8 -> 0.00 mm
- net Net-(Q1-E): track 13.1 -> 0.00 mm
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
Commit message: Final I hope
Other:
- outline, holes or cut-outs redrawn
