File: Digitronevé hod/LV part/Digitronove hodiny LV.kicad_pcb (KiCad board)
At the start: 2 copper layers, 27 parts, among them J10 Output, J11 Output, J12 RCWL-0516, J13 Output, J3 Output, J4 9V to 170V, J5 Output, J6 Output, J7 Output, J8 Output, J9 Output, SW1 RESET, SW2 SWITCH, SW3 +1, SW4 START/STOP, U2 DD4012SA

Commit message: Update Schéma LV
Parts:
- removed J4: 9V to 170V, Connector_PinHeader_1.00mm:PinHeader_1x03_P1.00mm_Horizontal
- removed J5: Output, Connector_PinHeader_1.00mm:PinHeader_1x01_P1.00mm_Horizontal
- added J1: ~, LOGIC-74HC595N_DIP16_:PDC004-PD, F.Cu at (269.0, 41.1)
- F1, F2: footprint Fuse:Fuseholder_Cylinder-5x20mm_Stelvio-Kontek_PTF78_Horizontal_Open -> Fuse:Fuse_1812_4532Metric
- J10: value Output -> GND; footprint Connector_PinHeader_1.00mm:PinHeader_1x01_P1.00mm_Horizontal -> Connector_PinHeader_1.00mm:PinHeader_1x01_P1.00mm_Vertical
- J11: value Output -> 5V; footprint Connector_PinHeader_1.00mm:PinHeader_1x01_P1.00mm_Horizontal -> Connector_PinHeader_1.00mm:PinHeader_1x01_P1.00mm_Vertical
- J12: value RCWL-0516 -> GND; footprint LOGIC-74HC595N_DIP16_:Untitled -> Connector_PinHeader_1.00mm:PinHeader_1x01_P1.00mm_Vertical
- J13: value Output -> RCWL-0516; footprint LOGIC-74HC595N_DIP16_:MAX1771 -> LOGIC-74HC595N_DIP16_:Untitled
- J2: value ~ -> 3V3; footprint LOGIC-74HC595N_DIP16_:PDC004-PD -> Connector_PinHeader_1.00mm:PinHeader_1x01_P1.00mm_Vertical
- J3: value Output -> MAX1771 module; footprint Connector_PinHeader_1.00mm:PinHeader_1x01_P1.00mm_Horizontal -> LOGIC-74HC595N_DIP16_:MAX1771
- J6: footprint Connector_PinHeader_1.00mm:PinHeader_1x01_P1.00mm_Horizontal -> Connector_PinHeader_1.00mm:PinHeader_1x01_P1.00mm_Vertical
- J7: value Output -> DATA; footprint Connector_PinHeader_1.00mm:PinHeader_1x01_P1.00mm_Horizontal -> Connector_PinHeader_1.00mm:PinHeader_1x01_P1.00mm_Vertical
- J8: value Output -> LATCH; footprint Connector_PinHeader_1.00mm:PinHeader_1x01_P1.00mm_Horizontal -> Connector_PinHeader_1.00mm:PinHeader_1x01_P1.00mm_Vertical
- J9: value Output -> STRL; footprint Connector_PinHeader_1.00mm:PinHeader_1x01_P1.00mm_Horizontal -> Connector_PinHeader_1.00mm:PinHeader_1x01_P1.00mm_Vertical
- U1: value ~ -> DD4012SA; footprint LOGIC-74HC595N_DIP16_:MODULE_ESP32_DEVKIT_V1 -> LOGIC-74HC595N_DIP16_:Untitled_3
- U2: value DD4012SA -> ~; footprint Converter_DCDC:Converter_DCDC_Murata_OKI-78SR_Horizontal -> LOGIC-74HC595N_DIP16_:MODULE_ESP32_DEVKIT_V1
- moved D1 176.4 mm to (243.8, 46.2), turned to 180 degrees
- moved R5 174.4 mm to (245.0, 87.5)
- moved F2 172.4 mm to (252.5, 38.6), turned to 180 degrees
- moved R6 171.0 mm to (244.0, 103.6), turned to 90 degrees
- moved F1 164.4 mm to (252.5, 43.6), turned to 180 degrees
- moved U2 154.0 mm to (234.7, 67.7), turned to 90 degrees
- moved R4 150.6 mm to (201.3, 42.1), turned to 180 degrees
- moved R1 146.2 mm to (201.3, 38.2), turned to 180 degrees
- moved R3 144.5 mm to (201.3, 49.7), turned to 180 degrees
- moved R2 144.4 mm to (201.3, 45.9), turned to 180 degrees
- moved U1 137.6 mm to (220.5, 42.5), turned to 90 degrees
- moved J12 136.3 mm to (258.0, 113.5)
- moved J3 128.8 mm to (263.0, 100.2), turned to 180 degrees
- moved J9 124.7 mm to (258.0, 117.5)
- moved J7 124.2 mm to (255.0, 117.5)
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Connections:
- D1 pad 1: Net-(D1-K) -> /5V
- D1 pad 2: Net-(D1-A) -> /5V
- F1 pad 1: Net-(U2-IN) -> /9V
- F1 pad 2: Net-(J2-Pin_2) -> /9V
- F2 pad 1: Net-(J4-Pin_1) -> /9V
- F2 pad 2: Net-(J2-Pin_2) -> /9V
- J10 pad 1: Net-(D1-A) -> GND
- J11 pad 1: GND -> /5V
- J2 pad 1: GND -> /3V3
- J9 pad 1: GND -> Net-(J9-Pin_1)
- R1 pad 1: Net-(J3-Pin_1) -> /3V3
- R1 pad 2: Net-(U1-EN) -> /3V3
- R2 pad 1: Net-(J3-Pin_1) -> /3V3
- R2 pad 2: Net-(U1-D33) -> /3V3
- R3 pad 1: Net-(J3-Pin_1) -> /3V3
- R3 pad 2: Net-(U1-D32) -> /3V3
- R4 pad 1: Net-(J3-Pin_1) -> /3V3
- R4 pad 2: Net-(U1-D27) -> /3V3
- R5 pad 1: Net-(U1-D2) -> /SHDN
- R5 pad 2: Net-(J4-Pin_3) -> /SHDN
- R6 pad 1: Net-(J5-Pin_1) -> Net-(J6-Pin_1)
- R6 pad 2: Net-(U1-D22) -> Net-(U2-D22)
- SW1 pad 2: Net-(U1-EN) -> /3V3
- SW2 pad 1: unconnected-(SW2-Pad1) -> GND
- SW2 pad 2: Net-(U1-D27) -> /3V3
- SW3 pad 2: Net-(U1-D32) -> /3V3
- SW4 pad 2: Net-(U1-D33) -> /3V3
- U1 pad 1: Net-(J3-Pin_1) -> /9V
- U1 pad 3: unconnected-(U1-D15-Pad3) -> /5V
- U2 pad 1: Net-(U2-IN) -> /3V3
- U2 pad 3: Net-(D1-A) -> unconnected-(U2-D15-Pad3)
Routing:
- net /3V3: track 0.00 -> 315.6 mm, vias 0 -> 1
- net /5V: track 0.00 -> 191.4 mm
- net /9V: track 0.00 -> 111.4 mm
- net /SHDN: track 0.00 -> 42.0 mm
- net Net-(J13-Pin_3): track 0.00 -> 21.1 mm, vias 0 -> 2
- net Net-(U2-D22): track 0.00 -> 16.4 mm
- added copper zone on B.Cu, net GND
- added copper zone on F.Cu, net GND
Other:
- board outline added: 100 x 100 mm

Commit message: Dokončení LV
Parts:
- moved STRL 66.7 mm to (195.6, 94.0)
- moved J10 61.1 mm to (192.6, 90.0)
- moved J11 61.1 mm to (198.6, 90.0)
- moved J12 61.1 mm to (201.6, 90.0)
- moved J2 61.1 mm to (195.6, 90.0)
- moved OUTPUT 61.1 mm to (192.6, 94.0)
- moved DATA 58.3 mm to (201.6, 94.0)
- moved LATCH 58.3 mm to (198.6, 94.0)
- moved J3 19.1 mm to (266.6, 119.0), turned to -90 degrees
- moved R6 16.6 mm to (233.6, 90.6), turned to 0 degrees
- moved R5 11.3 mm to (233.7, 87.5)
- renumbered J7 to DATA, J8 to LATCH, J6 to OUTPUT, J9 to STRL
Connections:
- R1 pad 2: /3V3 -> /EN
- R2 pad 2: /3V3 -> /START/STOP
- R3 pad 2: /3V3 -> /+1
- R4 pad 2: /3V3 -> /SWITCH
- SW1 pad 2: /3V3 -> /EN
- SW2 pad 2: /3V3 -> /SWITCH
- SW3 pad 2: /3V3 -> /+1
- SW4 pad 2: /3V3 -> /START/STOP
- U2 pad 16: /3V3 -> /EN
- U2 pad 21: /3V3 -> /+1
- U2 pad 22: /3V3 -> /START/STOP
- U2 pad 25: /3V3 -> /SWITCH
Routing:
- net /3V3: track 315.6 -> 95.6 mm
- net Net-(J9-Pin_1): track 0.00 -> 146.0 mm
- net Net-(J8-Pin_1): track 0.00 -> 136.1 mm
- net /EN: track 0.00 -> 123.5 mm
- net /SWITCH: track 0.00 -> 92.0 mm
- net /START/STOP: track 0.00 -> 83.7 mm, vias 0 -> 1
- net /+1: track 0.00 -> 80.3 mm, vias 0 -> 1
- net Net-(J7-Pin_1): track 0.00 -> 67.8 mm
- net Net-(J6-Pin_1): track 0.00 -> 42.4 mm
- net /5V: track 191.4 -> 175.7 mm, vias 0 -> 1
- net /9V: track 111.4 -> 124.6 mm
- net /SHDN: track 42.0 -> 48.5 mm, vias 0 -> 1
- net Net-(U2-D22): track 16.4 -> 17.7 mm, vias 0 -> 1
- net Net-(J13-Pin_3): track 21.1 -> 21.0 mm, vias 2 -> 1

Commit message: LV update
Parts:
- removed the R2 at (201.3, 45.9)
- removed the R3 at (201.3, 49.7)
- added R5: 10k, Resistor_THT:R_Axial_DIN0207_L6.3mm_D2.5mm_P10.16mm_Horizontal, F.Cu at (202.3, 70.0)
- added R6: 10k, Resistor_THT:R_Axial_DIN0207_L6.3mm_D2.5mm_P10.16mm_Horizontal, F.Cu at (198.9, 70.0)
- moved SW2 34.0 mm to (185.6, 49.3), turned to -90 degrees
- moved R1 33.0 mm to (192.2, 70.0), turned to -90 degrees
- moved R4 28.6 mm to (195.5, 70.0), turned to -90 degrees
- moved SW3 23.3 mm to (185.6, 39.1), turned to -90 degrees
- moved SW4 13.9 mm to (185.6, 59.3), turned to -90 degrees
- moved SW1 10.7 mm to (181.0, 76.0)
- renumbered J12 to J10, J13 to J11, OUTPUT to J4, DATA to J5, LATCH to J6, STRL to J7, J10 to J8, J11 to J9, R5 to R2, R6 to R3
Connections:
- R1 pad 1: /3V3 -> /EN
- R1 pad 2: /EN -> GND
- R4 pad 1: /3V3 -> /SWITCH
- R4 pad 2: /SWITCH -> GND
- SW1 pad 1: GND -> /3V3
- SW2 pad 1: GND -> /START/STOP
- SW2 pad 2: /SWITCH -> /3V3
- SW3 pad 1: GND -> /+1
- SW3 pad 2: /+1 -> /3V3
- SW4 pad 1: GND -> /SWITCH
- SW4 pad 2: /START/STOP -> /3V3
Routing:
- net /EN: track 123.5 -> 83.5 mm
- net /SWITCH: track 92.0 -> 66.6 mm
- net /+1: track 80.3 -> 101.3 mm, vias 1 -> 0
- net /3V3: track 95.6 -> 104.7 mm, vias 1 -> 0
- net /START/STOP: track 83.7 -> 90.0 mm, vias 1 -> 0

Commit message: Redesign LV
Parts:
- added J12: DS1302, LOGIC-74HC595N_DIP16_:Untitled_1, F.Cu at (220.4, 80.9)
- J3: value MAX1771 module -> MAX1771
- U2: value ~ -> ESP32 DevKit
- moved J3 127.0 mm to (140.4, 104.9), turned to 0 degrees
- moved D1 83.7 mm to (202.3, 118.9), turned to 0 degrees
- moved SW3 82.1 mm to (253.0, 86.0), turned to 180 degrees
- moved SW2 81.2 mm to (253.0, 94.5), turned to 180 degrees
- moved J11 80.3 mm to (161.8, 70.6), turned to -90 degrees
- moved J1 79.7 mm to (234.2, 112.9), turned to 0 degrees
- moved R2 73.3 mm to (164.7, 112.3), turned to 180 degrees
- moved U1 70.4 mm to (221.4, 112.9), turned to 180 degrees
- moved SW4 69.8 mm to (253.0, 77.4), turned to 180 degrees
- moved R4 69.5 mm to (253.1, 108.9)
- moved SW1 69.2 mm to (246.5, 98.3), turned to 0 degrees
- moved R1 64.8 mm to (244.0, 108.9)
- moved R6 64.3 mm to (250.1, 108.9)
- moved F2 63.6 mm to (226.2, 96.5)
- moved F1 63.1 mm to (226.2, 100.9)
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Connections:
- R3 pad 2: Net-(U2-D22) -> Net-(U2-D2)
- R4 pad 1: /SWITCH -> /START/STOP
- R6 pad 1: /START/STOP -> /SWITCH
- SW2 pad 1: /START/STOP -> /SWITCH
- SW4 pad 1: /SWITCH -> /START/STOP
- U2 pad 14: Net-(U2-D22) -> Net-(J12-Pin_3)
- U2 pad 15: Net-(J5-Pin_1) -> /START/STOP
- U2 pad 22: /START/STOP -> /SWITCH
- U2 pad 25: /SWITCH -> Net-(J5-Pin_1)
- U2 pad 26: unconnected-(U2-D14-Pad26) -> Net-(J11-Pin_3)
- U2 pad 28: unconnected-(U2-D13-Pad28) -> /SHDN
- U2 pad 4: /SHDN -> Net-(U2-D2)
- U2 pad 5: Net-(J11-Pin_3) -> Net-(J12-Pin_5)
- U2 pad 9: unconnected-(U2-D18-Pad9) -> Net-(J12-Pin_3)
Routing:
- net Net-(J7-Pin_1): track 146.0 -> 12.3 mm
- net Net-(J6-Pin_1): track 136.1 -> 12.3 mm
- net /SWITCH: track 66.6 -> 153.8 mm
- net /5V: track 175.7 -> 107.0 mm, vias 1 -> 0
- net Net-(J5-Pin_1): track 67.8 -> 12.3 mm
- net /EN: track 83.5 -> 134.6 mm
- net /+1: track 101.3 -> 143.3 mm
- net Net-(J4-Pin_1): track 42.4 -> 3.25 mm
- net /SHDN: track 48.5 -> 14.3 mm, vias 1 -> 0
- net /3V3: track 104.7 -> 131.7 mm
- net Net-(J12-Pin_5): track 0.00 -> 19.6 mm
- net Net-(J12-Pin_3): track 0.00 -> 19.4 mm
- net Net-(U2-D22): track 17.7 -> 0.00 mm, vias 1 -> 0
- net Net-(J11-Pin_3): track 21.0 -> 32.4 mm
- net /9V: track 124.6 -> 113.9 mm, vias 0 -> 1
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Other:
- board size 100 x 100 mm -> 136 x 62 mm

Commit message: Před kontrolou
Parts:
- added C1: 470uF, Capacitor_THT:CP_Radial_D10.0mm_P5.00mm, F.Cu at (161.9, 106.8)
- J10: renamed from J5; footprint Connector_PinHeader_1.00mm:PinHeader_1x01_P1.00mm_Vertical -> Connector_PinHeader_2.00mm:PinHeader_1x01_P2.00mm_Vertical
- J11: renamed from J8; footprint Connector_PinHeader_1.00mm:PinHeader_1x01_P1.00mm_Vertical -> Connector_PinHeader_2.00mm:PinHeader_1x01_P2.00mm_Vertical
- J12: renamed from J10; footprint Connector_PinHeader_1.00mm:PinHeader_1x01_P1.00mm_Vertical -> Connector_PinHeader_2.00mm:PinHeader_1x01_P2.00mm_Vertical
- J5: renamed from J4; footprint Connector_PinHeader_1.00mm:PinHeader_1x01_P1.00mm_Vertical -> Connector_PinHeader_2.00mm:PinHeader_1x01_P2.00mm_Vertical
- J7: renamed from J6; footprint Connector_PinHeader_1.00mm:PinHeader_1x01_P1.00mm_Vertical -> Connector_PinHeader_2.00mm:PinHeader_1x01_P2.00mm_Vertical
- J8: renamed from J9; footprint Connector_PinHeader_1.00mm:PinHeader_1x01_P1.00mm_Vertical -> Connector_PinHeader_2.00mm:PinHeader_1x01_P2.00mm_Vertical
- J9: renamed from J7; footprint Connector_PinHeader_1.00mm:PinHeader_1x01_P1.00mm_Vertical -> Connector_PinHeader_2.00mm:PinHeader_1x01_P2.00mm_Vertical
- moved J11 17.4 mm to (157.7, 88.3)
- moved J12 17.4 mm to (161.0, 88.3)
- moved R2 1.94 mm to (164.7, 114.2)
- renumbered J12 to J1, J1 to J2, J2 to J3, J3 to J4, J11 to J6, R6 to R4, R4 to R6
Routing:
- net /5V: track 107.0 -> 128.5 mm
- net Net-(J6-Pin_3): track 32.4 -> 43.7 mm, vias 1 -> 0
- net /9V: track 113.9 -> 119.1 mm
- net /SHDN: track 14.3 -> 17.2 mm
- net GND: vias 0 -> 5

Commit message: PCB finnal
Parts:
- added H1: MountingHole, MountingHole:MountingHole_2.5mm, F.Cu at (124.1, 68.4)
- added H2: MountingHole, MountingHole:MountingHole_2.5mm, F.Cu at (253.1, 68.4)
- added H3: MountingHole, MountingHole:MountingHole_2.5mm, F.Cu at (194.6, 123.4)
- J3: footprint Connector_PinHeader_1.00mm:PinHeader_1x01_P1.00mm_Vertical -> Connector_PinHeader_2.00mm:PinHeader_1x01_P2.00mm_Vertical
- moved R2 10.3 mm to (154.4, 114.2), turned to 0 degrees
- moved J8 6.16 mm to (198.4, 112.8)
- moved J3 2.89 mm to (208.2, 95.6), turned to 0 degrees
- moved R6 1.74 mm to (253.2, 110.6)
- moved R4 1.74 mm to (250.2, 110.6)
- moved R5 1.74 mm to (247.1, 110.6)
- moved R1 1.74 mm to (244.1, 110.6)
- moved J5 0.15 mm to (211.3, 106.0)
- moved D1 0.10 mm to (202.3, 119.0)
- moved R3 0.06 mm to (211.3, 102.6)
Routing:
- net /9V: track 119.1 -> 114.5 mm
- net /3V3: track 131.7 -> 135.7 mm
- net /START/STOP: track 99.1 -> 100.1 mm
- net /+1: track 143.3 -> 144.2 mm
- net /EN: track 134.6 -> 135.3 mm
- net /SWITCH: track 153.5 -> 154.3 mm
- net /5V: track 128.5 -> 128.0 mm
Other:
- outline, holes or cut-outs redrawn

Commit message: pcb uprava
Parts:
- removed J10: DATA, Connector_PinHeader_2.00mm:PinHeader_1x01_P2.00mm_Vertical
- removed J11, J12: GND, Connector_PinHeader_2.00mm:PinHeader_1x01_P2.00mm_Vertical
- removed J3: 3V3, Connector_PinHeader_2.00mm:PinHeader_1x01_P2.00mm_Vertical
- removed J5: Output, Connector_PinHeader_2.00mm:PinHeader_1x01_P2.00mm_Vertical
- removed J6: RCWL-0516, LOGIC-74HC595N_DIP16_:Untitled
- removed J7: LATCH, Connector_PinHeader_2.00mm:PinHeader_1x01_P2.00mm_Vertical
- removed J8: 5V, Connector_PinHeader_2.00mm:PinHeader_1x01_P2.00mm_Vertical
- removed J9: STRL, Connector_PinHeader_2.00mm:PinHeader_1x01_P2.00mm_Vertical
- added C2: 100nF, Capacitor_SMD:C_1206_3216Metric_Pad1.33x1.80mm_HandSolder, F.Cu at (170.4, 84.5)
- added C3: 100nF, Capacitor_SMD:C_1206_3216Metric_Pad1.33x1.80mm_HandSolder, F.Cu at (178.3, 84.5)
- added C4: 100nF, Capacitor_SMD:C_1206_3216Metric_Pad1.33x1.80mm_HandSolder, F.Cu at (186.2, 84.5)
- added DS1: Conn_01x06, LOGIC-74HC595N_DIP16_:DS3231, F.Cu at (236.8, 82.4)
- added Konektor1: Conn_01x09, Connector_JST:JST_EH_B9B-EH-A_1x09_P2.50mm_Vertical, F.Cu at (123.3, 94.4)
- added R10: 4.7k, Resistor_SMD:R_1206_3216Metric_Pad1.30x1.75mm_HandSolder, F.Cu at (177.0, 80.6)
- added R11: 4.7k, Resistor_SMD:R_1206_3216Metric_Pad1.30x1.75mm_HandSolder, F.Cu at (184.9, 80.6)
- added R7: 4.7k, Resistor_SMD:R_1206_3216Metric_Pad1.30x1.75mm_HandSolder, F.Cu at (169.1, 80.6)
- added R8: 4.7k, Resistor_SMD:R_1206_3216Metric_Pad1.30x1.75mm_HandSolder, F.Cu at (179.6, 80.6)
- added R9: 4.7k, Resistor_SMD:R_1206_3216Metric_Pad1.30x1.75mm_HandSolder, F.Cu at (187.4, 80.6)
- C1: value 470uF -> 100uF; footprint Capacitor_THT:CP_Radial_D10.0mm_P5.00mm -> Capacitor_THT:CP_Radial_D6.3mm_P2.50mm
- J1: value DS1302 -> ~; footprint LOGIC-74HC595N_DIP16_:Untitled_1 -> LOGIC-74HC595N_DIP16_:PDC004-PD
- J2: value ~ -> MAX1771; footprint LOGIC-74HC595N_DIP16_:PDC004-PD -> LOGIC-74HC595N_DIP16_:MAX1771
- J4: value MAX1771 -> GY-VL53L0X; footprint LOGIC-74HC595N_DIP16_:MAX1771 -> LOGIC-74HC595N_DIP16_:GY-VL53L0X
- R1: footprint Resistor_THT:R_Axial_DIN0207_L6.3mm_D2.5mm_P10.16mm_Horizontal -> Resistor_SMD:R_1206_3216Metric_Pad1.30x1.75mm_HandSolder
- R2, R4, R6: value 10k -> 4.7k; footprint Resistor_THT:R_Axial_DIN0207_L6.3mm_D2.5mm_P10.16mm_Horizontal -> Resistor_SMD:R_1206_3216Metric_Pad1.30x1.75mm_HandSolder
- R3: value 4.7k -> 10k; footprint Resistor_THT:R_Axial_DIN0207_L6.3mm_D2.5mm_P10.16mm_Horizontal -> Resistor_SMD:R_1206_3216Metric_Pad1.30x1.75mm_HandSolder; moved to B.Cu
- R5: value 10k -> 4.7k; footprint Resistor_THT:R_Axial_DIN0207_L6.3mm_D2.5mm_P10.16mm_Horizontal -> Resistor_SMD:R_1206_3216Metric_Pad1.30x1.75mm_HandSolder; moved to B.Cu
- SW1: value RESET -> START/STOP
- SW2: value SWITCH -> EN
- SW4: value START/STOP -> SWITCH
- moved R5 118.7 mm to (129.5, 94.4), turned to 0 degrees
- moved SW2 95.9 mm to (159.3, 74.5), turned to 90 degrees
- moved R6 86.9 mm to (171.7, 80.6), turned to 90 degrees
- moved SW1 82.9 mm to (167.1, 74.5), turned to 90 degrees
- moved SW3 78.8 mm to (175.1, 74.4), turned to 90 degrees
- moved SW4 70.1 mm to (182.9, 74.4), turned to 90 degrees
- moved R2 62.0 mm to (208.3, 83.4), turned to 90 degrees
- moved J4 51.2 mm to (191.0, 112.6)
- moved R1 48.9 mm to (203.4, 83.4), turned to 90 degrees
- moved R4 45.8 mm to (213.3, 83.4)
- moved U2 38.8 mm to (147.0, 112.1), turned to -90 degrees
- moved J1 37.6 mm to (224.8, 118.2)
- moved C1 21.4 mm to (177.8, 121.1), turned to -90 degrees
- moved R3 16.3 mm to (227.6, 103.8), turned to 0 degrees
- moved J2 9.35 mm to (243.4, 111.3), turned to 180 degrees
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Connections:
- net /5V renamed /+5V
- F1 pad 1: /9V -> /+9V
- F1 pad 2: /9V -> /+9V
- F2 pad 1: /9V -> /+9V
- F2 pad 2: /9V -> /+9V
- R1 pad 1: /EN -> /+3V3
- R1 pad 2: GND -> /SQW
- R2 pad 1: /SHDN -> /+3V3
- R2 pad 2: /SHDN -> /SCL
- R3 pad 1: Net-(J5-Pin_1) -> /SHDN
- R3 pad 2: Net-(U2-D2) -> /SHDN
- R4 pad 1: /SWITCH -> /SDA
- R4 pad 2: GND -> /+3V3
- R5 pad 1: /+1 -> /NE1,2
- R5 pad 2: GND -> /NE1,2
- R6 pad 1: /START/STOP -> /+3V3
- R6 pad 2: GND -> /+3V3
- SW1 pad 1: /3V3 -> GND
- SW1 pad 2: /EN -> /+3V3
- SW2 pad 1: /SWITCH -> GND
- SW2 pad 2: /3V3 -> /EN
- SW3 pad 1: /+1 -> GND
- SW3 pad 2: /3V3 -> /+3V3
- SW4 pad 1: /START/STOP -> GND
- SW4 pad 2: /3V3 -> /+3V3
- U1 pad 1: /9V -> /+9V
- U2 pad 1: /3V3 -> /+3V3
- U2 pad 14: Net-(J1-Pin_3) -> /OE
- U2 pad 15: /START/STOP -> /START-STOP
- U2 pad 20: unconnected-(U2-D35-Pad20) -> /SQW
- U2 pad 23: Net-(J7-Pin_1) -> /RLCK
- U2 pad 24: Net-(J9-Pin_1) -> /SRLCK
- U2 pad 25: Net-(J10-Pin_1) -> /SER1
- U2 pad 26: Net-(J6-Pin_3) -> unconnected-(U2-D14-Pad26)
- U2 pad 4: Net-(U2-D2) -> /NE1,2
- U2 pad 5: Net-(J1-Pin_5) -> /SCL
- U2 pad 9: Net-(J1-Pin_3) -> /SDA
Routing:
- net /+3V3: track 0.00 -> 204.0 mm, vias 0 -> 7
- net /3V3: track 135.7 -> 0.00 mm
- net /9V: track 114.5 -> 0.00 mm, vias 1 -> 0
- net /SQW: track 0.00 -> 109.3 mm, vias 0 -> 3
- net /SDA: track 0.00 -> 103.5 mm, vias 0 -> 1
- net /START/STOP: track 100.1 -> 0.00 mm
- net /SCL: track 0.00 -> 93.2 mm, vias 0 -> 1
- net /SER1: track 0.00 -> 87.8 mm
- net /RLCK: track 0.00 -> 85.0 mm, vias 0 -> 1
- net /SRLCK: track 0.00 -> 84.3 mm, vias 0 -> 1
- net /SWITCH: track 154.3 -> 79.2 mm, vias 0 -> 2
- net /+1: track 144.2 -> 73.4 mm, vias 0 -> 2
- net /SHDN: track 17.0 -> 86.3 mm
- net /START-STOP: track 0.00 -> 60.8 mm, vias 0 -> 2
- net /EN: track 135.3 -> 84.9 mm, vias 0 -> 2
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
Commit message: Final I hope
Parts:
- J4: value GY-VL53L0X -> RCWL-0516
- moved J4 3.18 mm to (188.2, 111.1)
Routing:
- net /+3V3: track 204.0 -> 199.6 mm
- net /SDA: track 103.5 -> 99.7 mm
- net /SCL: track 93.2 -> 89.3 mm
Changed lines of the file:
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@@
 			(outputformat 1)
 			(mirror no)
-			(drillshape 1)
+			(drillshape 0)
 			(scaleselection 1)
-			(outputdirectory "")
+			(outputdirectory "dolnideska/")
 		)
 	)
@@
 	(footprint "LOGIC-74HC595N_DIP16_:GY-VL53L0X"
 		(layer "F.Cu")
-		(at 190.984 112.6472)
+		(at 188.19 111.1232)
 		(property "Reference" "J4"
 			(at 7.255 13.914 0)
@@
 			)
 		)
-		(property "Value" "GY-VL53L0X"
+		(property "Value" "RCWL-0516"
 			(at 7.255 15.414 0)
 			(unlocked yes)
@@
 		)
 		(fp_rect
-			(start 0.254 -0.508)
-			(end 4.064 4.572)
+			(start 0.254 -0.254)
+			(end 3.81 4.826)
 			(stroke
 				(width 0.1)
@@
 			(pintype "passive")
 		)
+		(pad "B" thru_hole circle
+			(at 5.334 3.81)
+			(size 2 2)
+			(drill 1)
+			(layers "*.Cu" "*.Mask")
+			(remove_unused_layers no)
+		)
 		(pad "GND" thru_hole circle
 			(at -5.08 -1.27)
@@
 			(pintype "passive")
 		)
+		(pad "X" thru_hole circle
+			(at 5.334 1.27)
+			(size 2 2)
+			(drill 1)
+			(layers "*.Cu" "*.Mask")
+			(remove_unused_layers no)
+		)
 		(embedded_fonts no)
 	)
@@
 	)
 	(segment
-		(start 210.008 80.1352)
-		(end 208.256 81.8872)
+		(start 183.11 112.3932)
+		(end 205.996 89.5072)
 		(width 0.4)
 		(layer "F.Cu")
@@
 	)
 	(segment
-		(start 159.869 106.9322)
-		(end 166.8864 113.9496)
+		(start 210.008 80.1352)
+		(end 208.256 81.8872)
 		(width 0.4)
 		(layer "F.Cu")
@@
 	)
 	(segment
-		(start 219.431 81.1412)
-		(end 218.152 81.1412)
+		(start 165.33 112.3932)
+		(end 183.11 112.3932)
 		(width 0.4)
 		(layer "F.Cu")
@@
 	)
 	(segment
-		(start 166.8864 113.9496)
-		(end 185.8716 113.9496)
+		(start 219.431 81.1412)
+		(end 218.152 81.1412)
 		(width 0.4)
 		(layer "F.Cu")
@@
 	)
 	(segment
-		(start 185.8716 113.9496)
-		(end 205.996 93.8252)
+		(start 159.869 106.9322)
+		(end 165.33 112.3932)
 		(width 0.4)
 		(layer "F.Cu")
@@
 	)
 	(segment
-		(start 205.996 93.8252)
+		(start 205.996 89.5072)
 		(end 205.996 84.1472)
 		(width 0.4)
@@
 	)
 	(segment
-		(start 205.996 84.1472)
-		(end 208.256 81.8872)
+		(start 218.152 81.1412)
+		(end 217.146 80.1352)
 		(width 0.4)
 		(layer "F.Cu")
@@
 	)
 	(segment
-		(start 218.152 81.1412)
-		(end 217.146 80.1352)
+		(start 217.146 80.1352)
+		(end 210.008 80.1352)
 		(width 0.4)
 		(layer "F.Cu")
@@
 	)
 	(segment
-		(start 217.146 80.1352)
-		(end 210.008 80.1352)
+		(start 205.996 84.1472)
+		(end 208.256 81.8872)
 		(width 0.4)
 		(layer "F.Cu")
@@
 	)
 	(segment
-		(start 210.822 91.5392)
-		(end 185.8716 116.4896)
+		(start 183.11 114.9332)
+		(end 166.092 114.9332)
 		(width 0.4)
 		(layer "F.Cu")
@@
 	(segment
 		(start 213.336 81.8872)
-		(end 216.612 81.8872)
+		(end 210.822 84.4012)
 		(width 0.4)
 		(layer "F.Cu")
@@
 	(segment
 		(start 213.336 81.8872)
-		(end 210.822 84.4012)
+		(end 216.612 81.8872)
 		(width 0.4)
 		(layer "F.Cu")
@@
 	(segment
 		(start 210.822 84.4012)
-		(end 210.822 91.5392)
+		(end 210.822 87.2212)
 		(width 0.4)
 		(layer "F.Cu")
@@
 	)
 	(segment
-		(start 185.8716 116.4896)
-		(end 167.6484 116.4896)
+		(start 210.822 87.2212)
+		(end 183.11 114.9332)
 		(width 0.4)
 		(layer "F.Cu")
@@
 	)
 	(segment
-		(start 167.6484 116.4896)
-		(end 158.726 107.5672)
+		(start 216.612 81.8872)
+		(end 218.406 83.6812)
 		(width 0.4)
 		(layer "F.Cu")
@@
 	)
 	(segment
-		(start 216.612 81.8872)
-		(end 218.406 83.6812)
+		(start 166.092 114.9332)
+		(end 158.726 107.5672)
 		(width 0.4)
 		(layer "F.Cu")
@@
 	)
 	(segment
+		(start 176.506 90.8032)
+		(end 166.6 90.8032)
+		(width 0.5)
+		(layer "F.Cu")
+		(net 28)
+	)
+	(segment
 		(start 165.33 88.7712)
 		(end 165.33 90.2952)
@@
 	)
 	(segment
-		(start 187.454 82.1672)
-		(end 187.428 82.1932)
+		(start 183.11 107.3132)
+		(end 179.554 107.3132)
 		(width 0.5)
 		(layer "F.Cu")
@@
 	)
 	(segment
-		(start 185.904 108.8372)
-		(end 179.4143 108.8372)
+		(start 187.454 82.1672)
+		(end 187.428 82.1932)
 		(width 0.5)
 		(layer "F.Cu")
@@
 	)
 	(segment
-		(start 178.577 107.9999)
-		(end 178.577 92.8742)
+		(start 179.554 107.3132)
+		(end 178.577 106.3362)
 		(width 0.5)
 		(layer "F.Cu")
@@
 	)
 	(segment
-		(start 179.4143 108.8372)
-		(end 178.577 107.9999)
-		(width 0.5)
-		(layer "F.Cu")
-		(net 28)
-	)
-	(segment
 		(start 178.577 92.8742)
 		(end 176.506 90.8032)
@@
 	)
 	(segment
-		(start 166.6 90.8032)
-		(end 165.33 92.0732)
-		(width 0.5)
-		(layer "F.Cu")
-		(net 28)
-	)
-	(segment
-		(start 176.506 90.8032)
-		(end 166.6 90.8032)
+		(start 169.14 79.0932)
+		(end 171.68 79.0932)
 		(width 0.5)
 		(layer "F.Cu")
@@
 	)
 	(segment
-		(start 169.14 79.0932)
-		(end 171.68 79.0932)
+		(start 166.6 90.8032)
+		(end 165.33 92.0732)
 		(width 0.5)
 		(layer "F.Cu")
@@
 		(width 0.5)
 		(layer "F.Cu")
+		(net 28)
+	)
+	(segment
+		(start 178.577 106.3362)
+		(end 178.577 92.8742)
+		(width 0.5)
+		(layer "F.Cu")
