File: Digitronevé hod/LV part/Digitronove hodiny LV.kicad_sch (KiCad schematic)
At the start: 27 parts, among them J10 GND, J11 RCWL-0516, J12 DS1302, J2 3V3, J3 MAX1771, J4 Output, J5 DATA, J6 LATCH, J7 STRL, J8 GND, J9 5V, SW1 RESET, SW2 SWITCH, SW3 +1, SW4 START/STOP, U1 DD4012SA, U2 ESP32 DevKit

Commit message: Před kontrolou
Parts:
- added C1: 470uF, Capacitor_THT:CP_Radial_D10.0mm_P5.00mm, symbol Device:C
- J10: renamed from J5; footprint Connector_PinHeader_1.00mm:PinHeader_1x01_P1.00mm_Vertical -> Connector_PinHeader_2.00mm:PinHeader_1x01_P2.00mm_Vertical
- J11: renamed from J8; footprint Connector_PinHeader_1.00mm:PinHeader_1x01_P1.00mm_Vertical -> Connector_PinHeader_2.00mm:PinHeader_1x01_P2.00mm_Vertical
- J12: renamed from J10; footprint Connector_PinHeader_1.00mm:PinHeader_1x01_P1.00mm_Vertical -> Connector_PinHeader_2.00mm:PinHeader_1x01_P2.00mm_Vertical
- J5: renamed from J4; footprint Connector_PinHeader_1.00mm:PinHeader_1x01_P1.00mm_Vertical -> Connector_PinHeader_2.00mm:PinHeader_1x01_P2.00mm_Vertical
- J7: renamed from J6; footprint Connector_PinHeader_1.00mm:PinHeader_1x01_P1.00mm_Vertical -> Connector_PinHeader_2.00mm:PinHeader_1x01_P2.00mm_Vertical
- J8: renamed from J9; footprint Connector_PinHeader_1.00mm:PinHeader_1x01_P1.00mm_Vertical -> Connector_PinHeader_2.00mm:PinHeader_1x01_P2.00mm_Vertical
- J9: renamed from J7; footprint Connector_PinHeader_1.00mm:PinHeader_1x01_P1.00mm_Vertical -> Connector_PinHeader_2.00mm:PinHeader_1x01_P2.00mm_Vertical
- renumbered J12 to J1, J1 to J2, J2 to J3, J3 to J4, J11 to J6, R6 to R4, R4 to R6
Connections:
- net 5V: now also C1.1
- net GND: now also C1.2
- no-connect marks 2 -> 15
Other:
- note removed: "GND"
- moved on the sheet: J11, J12, R1, R5, R6

Commit message: PCB finnal
Parts:
- added H1, H2, H3: MountingHole, MountingHole:MountingHole_2.5mm, symbol Mechanical:MountingHole
- J3: footprint Connector_PinHeader_1.00mm:PinHeader_1x01_P1.00mm_Vertical -> Connector_PinHeader_2.00mm:PinHeader_1x01_P2.00mm_Vertical
Changed lines of the file:
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@@
+	)
+	(symbol
+		(lib_id "Mechanical:MountingHole")
+		(at 66.04 114.3 0)
+		(unit 1)
+		(exclude_from_sim no)
+		(in_bom no)
+		(on_board yes)
+		(dnp no)
+		(fields_autoplaced yes)
+		(property "Reference" "H1"
+			(at 68.58 113.0299 0)
+			(effects
+				(font
+					(size 1.27 1.27)
+				)
+				(justify left)
+			)
+		)
+		(property "Value" "MountingHole"
+			(at 68.58 115.5699 0)
+			(effects
+				(font
+					(size 1.27 1.27)
+				)
+				(justify left)
+			)
+		)
+		(property "Footprint" "MountingHole:MountingHole_2.5mm"
+			(at 66.04 114.3 0)
+			(effects
+				(font
+					(size 1.27 1.27)
+				)
+				(hide yes)
+			)
+		)
+		(property "Datasheet" "~"
+			(at 66.04 114.3 0)
+			(effects
+				(font
+					(size 1.27 1.27)
+				)
+				(hide yes)
+			)
+		)
+		(property "Description" "Mounting Hole without connection"
+			(at 66.04 114.3 0)
+			(effects
+				(font
+					(size 1.27 1.27)
+				)
+				(hide yes)
+			)
+		)
+		(instances
+			(project "Digitronove hodiny LV"
+				(path "/760f652f-b82b-45ad-92c5-42c0d0511f5b"
+					(reference "H1")
+					(unit 1)
+				)
+			)
+		)
 	)
 	(symbol
@@
 	)
 	(symbol
+		(lib_id "Mechanical:MountingHole")
+		(at 66.04 123.19 0)
+		(unit 1)
+		(exclude_from_sim no)
+		(in_bom no)
+		(on_board yes)
+		(dnp no)
+		(fields_autoplaced yes)
+		(property "Reference" "H2"
+			(at 68.58 121.9199 0)
+			(effects
+				(font
+					(size 1.27 1.27)
+				)
+				(justify left)
+			)
+		)
+		(property "Value" "MountingHole"
+			(at 68.58 124.4599 0)
+			(effects
+				(font
+					(size 1.27 1.27)
+				)
+				(justify left)
+			)
+		)
+		(property "Footprint" "MountingHole:MountingHole_2.5mm"
+			(at 66.04 123.19 0)
+			(effects
+				(font
+					(size 1.27 1.27)
+				)
+				(hide yes)
+			)
+		)
+		(property "Datasheet" "~"
+			(at 66.04 123.19 0)
+			(effects
+				(font
+					(size 1.27 1.27)
+				)
+				(hide yes)
+			)
+		)
+		(property "Description" "Mounting Hole without connection"
+			(at 66.04 123.19 0)
+			(effects
+				(font
+					(size 1.27 1.27)
+				)
+				(hide yes)
+			)
+		)
+		(instances
+			(project "Digitronove hodiny LV"
+				(path "/760f652f-b82b-45ad-92c5-42c0d0511f5b"
+					(reference "H2")
+					(unit 1)
+				)
+			)
+		)
+	)
+	(symbol
 		(lib_id "Connector_Generic:Conn_01x03")
 		(at 274.32 82.55 0)
@@
 			)
 		)
-		(property "Footprint" "Connector_PinHeader_1.00mm:PinHeader_1x01_P1.00mm_Vertical"
+		(property "Footprint" "Connector_PinHeader_2.00mm:PinHeader_1x01_P2.00mm_Vertical"
 			(at 152.4 71.12 0)
 			(effects
@@
 					(unit 1)
 				)
+			)
+		)
+	)
+	(symbol
+		(lib_id "Mechanical:MountingHole")
+		(at 66.04 132.08 0)
+		(unit 1)
+		(exclude_from_sim no)
+		(in_bom no)
+		(on_board yes)
+		(dnp no)
+		(fields_autoplaced yes)
+		(property "Reference" "H3"
+			(at 68.58 130.8099 0)
+			(effects
+				(font
+					(size 1.27 1.27)
+				)
+				(justify left)
+			)
+		)
+		(property "Value" "MountingHole"
+			(at 68.58 133.3499 0)
+			(effects
+				(font
+					(size 1.27 1.27)
+				)
+				(justify left)
+			)
+		)
+		(property "Footprint" "MountingHole:MountingHole_2.5mm"
+			(at 66.04 132.08 0)
+			(effects
+				(font
+					(size 1.27 1.27)
+				)
+				(hide yes)
+			)
+		)
+		(property "Datasheet" "~"
+			(at 66.04 132.08 0)
+			(effects
+				(font
+					(size 1.27 1.27)
+				)
+				(hide yes)
+			)
+		)
+		(property "Description" "Mounting Hole without connection"
+			(at 66.04 132.08 0)
+			(effects
+				(font
+					(size 1.27 1.27)
+				)
+				(hide yes)
+			)
+		)
+		(instances
+			(project "Digitronove hodiny LV"
+				(path "/760f652f-b82b-45ad-92c5-42c0d0511f5b"
+					(reference "H3")
+					(unit 1)
+				)

Commit message: pcb uprava
Parts:
- removed J1: DS1302, LOGIC-74HC595N_DIP16_:Untitled_1, symbol Connector_Generic:Conn_01x05
- removed J10: DATA, Connector_PinHeader_2.00mm:PinHeader_1x01_P2.00mm_Vertical, symbol Connector_Generic:Conn_01x01
- removed J11, J12: GND, Connector_PinHeader_2.00mm:PinHeader_1x01_P2.00mm_Vertical, symbol Connector_Generic:Conn_01x01
- removed J3: 3V3, Connector_PinHeader_2.00mm:PinHeader_1x01_P2.00mm_Vertical, symbol Connector_Generic:Conn_01x01
- removed J5: Output, Connector_PinHeader_2.00mm:PinHeader_1x01_P2.00mm_Vertical, symbol Connector_Generic:Conn_01x01
- removed J6: RCWL-0516, LOGIC-74HC595N_DIP16_:Untitled, symbol Connector_Generic:Conn_01x05
- removed J7: LATCH, Connector_PinHeader_2.00mm:PinHeader_1x01_P2.00mm_Vertical, symbol Connector_Generic:Conn_01x01
- removed J8: 5V, Connector_PinHeader_2.00mm:PinHeader_1x01_P2.00mm_Vertical, symbol Connector_Generic:Conn_01x01
- removed J9: STRL, Connector_PinHeader_2.00mm:PinHeader_1x01_P2.00mm_Vertical, symbol Connector_Generic:Conn_01x01
- removed R5: 10k, Resistor_THT:R_Axial_DIN0207_L6.3mm_D2.5mm_P10.16mm_Horizontal, symbol Device:R
- added C2, C3, C4: 100nF, Capacitor_SMD:C_1206_3216Metric_Pad1.33x1.80mm_HandSolder, symbol Device:C
- added DS1: Conn_01x06, LOGIC-74HC595N_DIP16_:DS3231, symbol Connector_Generic:Conn_01x06
- added J4: GY-VL53L0X, LOGIC-74HC595N_DIP16_:GY-VL53L0X, symbol Connector_Generic:Conn_01x04
- added Konektor1: Conn_01x09, Connector_JST:JST_EH_B9B-EH-A_1x09_P2.50mm_Vertical, symbol Connector_Generic:Conn_01x09
- added R10, R11, R2, R7, R8, R9: 4.7k, Resistor_SMD:R_1206_3216Metric_Pad1.30x1.75mm_HandSolder, symbol Device:R
- C1: value 470uF -> 100uF; footprint Capacitor_THT:CP_Radial_D10.0mm_P5.00mm -> Capacitor_THT:CP_Radial_D6.3mm_P2.50mm
- R1: footprint Resistor_THT:R_Axial_DIN0207_L6.3mm_D2.5mm_P10.16mm_Horizontal -> Resistor_SMD:R_1206_3216Metric_Pad1.30x1.75mm_HandSolder
- R3: renamed from R2; footprint Resistor_THT:R_Axial_DIN0207_L6.3mm_D2.5mm_P10.16mm_Horizontal -> Resistor_SMD:R_1206_3216Metric_Pad1.30x1.75mm_HandSolder
- R4, R6: value 10k -> 4.7k; footprint Resistor_THT:R_Axial_DIN0207_L6.3mm_D2.5mm_P10.16mm_Horizontal -> Resistor_SMD:R_1206_3216Metric_Pad1.30x1.75mm_HandSolder
- R5: renamed from R3; footprint Resistor_THT:R_Axial_DIN0207_L6.3mm_D2.5mm_P10.16mm_Horizontal -> Resistor_SMD:R_1206_3216Metric_Pad1.30x1.75mm_HandSolder
- SW1: value RESET -> START/STOP
- SW2: value SWITCH -> EN
- SW4: value START/STOP -> SWITCH
- renumbered J2 to J1, J4 to J2
Connections:
- net +1: now also C3.2, R10.2; no longer SW3.1
- net EN: now also SW2.2; no longer R1.1, SW1.2
- net GND: now also SW1.1, SW2.1, SW3.1, SW4.1, C2.1, C3.1, C4.1, DS1.GND, J4.GND, Konektor1.4 (Pin_4), Konektor1.5 (Pin_5); no longer R1.2, R4.2, R6.2
- net SWITCH: now also C4.2, R11.2; no longer R4.1, SW2.1
- net SRLCK: now reaches U2.24 (D26)
- net SRLCK: now also Konektor1.6 (Pin_6)
- net OE: now reaches U2.14 (D22)
- net OE: now also Konektor1.8 (Pin_8); no longer U2.9 (D18)
- net SCL: now reaches U2.5 (D4)
- net SCL: now also DS1.SCL, J4.SCL, R2.2
- net SER1: now reaches U2.25 (D27)
- net SER1: now also Konektor1.9 (Pin_9)
- net NE1,2: now reaches R5.1
- net NE1,2: now also R5.2, U2.4 (D2), Konektor1.1 (Pin_1)
- net RLCK: now reaches U2.23 (D25)
- net RLCK: now also Konektor1.7 (Pin_7)
- net SQW: now reaches U2.20 (D35)
- net SQW: now also R1.2, DS1.SQW
- net 3V3 renamed +3V3
- net +3V3: now also R1.1, R4.2, R6.1, R6.2, SW1.2, DS1.+3V3, J4.+3V3, Konektor1.3 (Pin_3), R10.1, R11.1, R2.1, R7.1, R8.1, R8.2, R9.1, R9.2; no longer SW1.1, SW2.2
- net 5V renamed +5V
- net +5V: now also Konektor1.2 (Pin_2)
- net 9V renamed +9V
- removed net START/STOP: R6.1, SW4.1, U2.15 (D23)
- new net SDA: DS1.SDA, J4.SDA, R4.1, U2.9 (D18)
- new net START-STOP: C2.2, R7.2, U2.15 (D23)
- no-connect marks 15 -> 16
Other:
- note removed: "3V3 pro 595"
- note removed: "5V"
- note removed: "9V"
- note removed: "DATA/LATCH/STRL"
- note removed: "tečka"
- moved on the sheet: C1, D1, F1, F2, H1, H2, H3, J1, J2, R3, U1, U2

Commit message: Final I hope
Parts:
- added Q1: NPN, symbol Simulation_SPICE:NPN
Connections:
- net GND: now also Q1.3 (E)
- net SHDN: now also Q1.1 (C); no longer R3.2
- new net: Q1.2 (B), R3.2
Other:
- title: (none) -> Dolní deska
- moved on the sheet: R3
Changed lines of the file:
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@@
 	(generator_version "9.0")
 	(paper "A4")
+	(title_block
+		(title "Dolní deska")
+		(date "08.04.2025")
+	)
 	(text "USB-C s modulem Ip2721"
 		(exclude_from_sim no)
@@
 	(wire
 		(pts
-			(xy 160.02 101.6) (xy 205.74 101.6)
+			(xy 160.02 101.6) (xy 209.55 101.6)
 		)
 		(stroke
@@
 	(wire
 		(pts
-			(xy 205.74 82.55) (xy 226.06 82.55)
+			(xy 127 68.58) (xy 129.54 68.58)
 		)
 		(stroke
@@
 	(wire
 		(pts
-			(xy 127 68.58) (xy 129.54 68.58)
+			(xy 44.45 128.27) (xy 44.45 124.46)
 		)
 		(stroke
@@
 	(wire
 		(pts
-			(xy 44.45 128.27) (xy 44.45 124.46)
+			(xy 29.21 125.73) (xy 29.21 124.46)
 		)
 		(stroke
@@
 	(wire
 		(pts
-			(xy 29.21 125.73) (xy 29.21 124.46)
+			(xy 162.56 71.12) (xy 160.02 71.12)
 		)
 		(stroke
@@
 	(wire
 		(pts
-			(xy 162.56 71.12) (xy 160.02 71.12)
+			(xy 224.79 95.25) (xy 224.79 96.52)
 		)
 		(stroke
@@
 	(wire
 		(pts
+			(xy 240.03 82.55) (xy 241.3 82.55)
+		)
+		(stroke
+			(width 0)
+			(type default)
+		)
+	)
+	(wire
+		(pts
 			(xy 41.91 87.63) (xy 50.8 87.63)
 		)
@@
 	(wire
 		(pts
-			(xy 226.06 80.01) (xy 241.3 80.01)
-		)
-		(stroke
-			(width 0)
-			(type default)
-		)
-	)
-	(wire
-		(pts
 			(xy 162.56 109.22) (xy 160.02 109.22)
 		)
@@
 	(wire
 		(pts
-			(xy 223.52 77.47) (xy 226.06 77.47)
-		)
-		(stroke
-			(width 0)
-			(type default)
-		)
-	)
-	(wire
-		(pts
-			(xy 205.74 82.55) (xy 205.74 101.6)
-		)
-		(stroke
-			(width 0)
-			(type default)
-		)
-	)
-	(wire
-		(pts
-			(xy 226.06 77.47) (xy 226.06 80.01)
-		)
-		(stroke
-			(width 0)
-			(type default)
-		)
-	)
-	(wire
-		(pts
 			(xy 68.58 161.29) (xy 68.58 160.02)
 		)
@@
 	(wire
 		(pts
-			(xy 241.3 82.55) (xy 233.68 82.55)
+			(xy 45.72 38.1) (xy 43.18 38.1)
 		)
 		(stroke
@@
 	(wire
 		(pts
-			(xy 45.72 38.1) (xy 43.18 38.1)
+			(xy 45.72 48.26) (xy 43.18 48.26)
 		)
 		(stroke
@@
 	(wire
 		(pts
-			(xy 45.72 48.26) (xy 43.18 48.26)
+			(xy 231.14 80.01) (xy 241.3 80.01)
 		)
 		(stroke
@@
 	)
 	(label "SHDN"
-		(at 233.68 82.55 0)
+		(at 240.03 82.55 180)
 		(effects
 			(font
 				(size 1.27 1.27)
 			)
-			(justify left bottom)
+			(justify right bottom)
 		)
 	)
@@
 		)
 	)
+	(label "SHDN"
+		(at 224.79 95.25 180)
+		(effects
+			(font
+				(size 1.27 1.27)
+			)
+			(justify right bottom)
+		)
+	)
 	(label "NE1,2"
 		(at 45.72 35.56 0)
@@
 	(symbol
 		(lib_id "power:GND")
-		(at 223.52 77.47 0)
+		(at 231.14 80.01 0)
 		(unit 1)
 		(exclude_from_sim no)
@@
 		(dnp no)
 		(property "Reference" "#PWR06"
-			(at 223.52 83.82 0)
+			(at 231.14 86.36 0)
 			(effects
 				(font
@@
 		)
 		(property "Value" "GND"
-			(at 223.52 81.28 0)
+			(at 231.14 83.82 0)
 			(effects
 				(font
@@
 		)
 		(property "Footprint" ""
-			(at 223.52 77.47 0)
+			(at 231.14 80.01 0)
 			(effects
 				(font
@@
 		)
 		(property "Datasheet" ""
-			(at 223.52 77.47 0)
+			(at 231.14 80.01 0)
 			(effects
 				(font
@@
 		)
 		(property "Description" "Power symbol creates a global label with name \"GND\" , ground"
-			(at 223.52 77.47 0)
+			(at 231.14 80.01 0)
 			(effects
 				(font
@@
 	)
 	(symbol
+		(lib_id "power:GND")
+		(at 224.79 106.68 0)
+		(unit 1)
+		(exclude_from_sim no)
+		(in_bom yes)
+		(on_board yes)
+		(dnp no)
+		(property "Reference" "#PWR07"
+			(at 224.79 113.03 0)
+			(effects
+				(font
+					(size 1.27 1.27)
+				)
+				(hide yes)
+			)
+		)
+		(property "Value" "GND"
+			(at 224.79 110.49 0)
+			(effects
+				(font
+					(size 1.27 1.27)
+				)
+			)
+		)
+		(property "Footprint" ""
+			(at 224.79 106.68 0)
+			(effects
+				(font
+					(size 1.27 1.27)
+				)
+				(hide yes)
+			)
+		)
+		(property "Datasheet" ""
+			(at 224.79 106.68 0)
+			(effects
+				(font
+					(size 1.27 1.27)
+				)
+				(hide yes)
+			)
+		)
+		(property "Description" "Power symbol creates a global label with name \"GND\" , ground"
+			(at 224.79 106.68 0)
+			(effects
+				(font
+					(size 1.27 1.27)
+				)
+				(hide yes)
+			)
+		)
+		(pin "1"
+		)
+		(instances
+			(project "Digitronove hodiny LV"
+				(path "/760f652f-b82b-45ad-92c5-42c0d0511f5b"
+					(reference "#PWR07")
+					(unit 1)
+				)
+			)
+		)
+	)
+	(symbol
 		(lib_id "Switch:SW_Push")
 		(at 68.58 165.1 270)
@@
 	(symbol
 		(lib_id "Device:R")
-		(at 229.87 82.55 90)
+		(at 213.36 101.6 90)
 		(mirror x)
 		(unit 1)
@@
 		(dnp no)
 		(property "Reference" "R3"
-			(at 229.87 84.582 90)
+			(at 213.36 103.632 90)
 			(effects
 				(font
@@
 		)
 		(property "Value" "10k"
-			(at 229.87 82.55 90)
+			(at 213.36 101.6 90)
 			(effects
 				(font
@@
 		)
 		(property "Footprint" "Resistor_SMD:R_1206_3216Metric_Pad1.30x1.75mm_HandSolder"
-			(at 229.87 80.772 90)
+			(at 213.36 99.822 90)
 			(effects
 				(font
@@
 		)
 		(property "Datasheet" "~"
-			(at 229.87 82.55 0)
+			(at 213.36 101.6 0)
 			(effects
 				(font
@@
 		)
 		(property "Description" "Resistor"
-			(at 229.87 82.55 0)
+			(at 213.36 101.6 0)
 			(effects
 				(font
@@
 					(unit 1)
 				)
+			)
+		)
+	)
+	(symbol
+		(lib_id "Simulation_SPICE:NPN")
+		(at 222.25 101.6 0)
+		(unit 1)
+		(exclude_from_sim no)
+		(in_bom yes)
+		(on_board yes)
+		(dnp no)
+		(fields_autoplaced yes)
+		(property "Reference" "Q1"
+			(at 227.33 100.3299 0)
+			(effects
+				(font
+					(size 1.27 1.27)
+				)
+				(justify left)
+			)
+		)
+		(property "Value" "NPN"
+			(at 227.33 102.8699 0)
+			(effects
+				(font
+					(size 1.27 1.27)
+				)
+				(justify left)
+			)
+		)
+		(property "Footprint" ""
+			(at 285.75 101.6 0)
+			(effects
+				(font
+					(size 1.27 1.27)
+				)
+				(hide yes)
+			)
+		)
+		(property "Datasheet" "https://ngspice.sourceforge.io/docs/ngspice-html-manual/manual.xhtml#cha_BJTs"
+			(at 285.75 101.6 0)
+			(effects
+				(font
+					(size 1.27 1.27)
+				)
+				(hide yes)
+			)
+		)
+		(property "Description" "Bipolar transistor symbol for simulation only, substrate tied to the emitter"
+			(at 222.25 101.6 0)
+			(effects
+				(font
+					(size 1.27 1.27)
+				)
+				(hide yes)
+			)
+		)
+		(property "Sim.Device" "NPN"
+			(at 222.25 101.6 0)
+			(effects
+				(font
+					(size 1.27 1.27)
+				)
+				(hide yes)
+			)
+		)
+		(property "Sim.Type" "GUMMELPOON"
+			(at 222.25 101.6 0)
+			(effects
+				(font
+					(size 1.27 1.27)
+				)
+				(hide yes)
+			)
+		)
+		(property "Sim.Pins" "1=C 2=B 3=E"
+			(at 222.25 101.6 0)
+			(effects
+				(font
+					(size 1.27 1.27)
+				)
+				(hide yes)
+			)
+		)
+		(pin "1"
+		)
+		(pin "2"
+		)
+		(pin "3"
+		)
+		(instances
+			(project ""
+				(path "/760f652f-b82b-45ad-92c5-42c0d0511f5b"
+					(reference "Q1")
+					(unit 1)
+				)

Commit message: release meee
Other:
- title: Dolní deska -> Příloha I
Changed lines of the file:
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@@
 	(paper "A4")
 	(title_block
-		(title "Dolní deska")
+		(title "Příloha I")
 		(date "08.04.2025")
+		(rev "Augusta Jan")
+		(comment 1 "Dolní PCB")
 	)
 	(text "USB-C s modulem Ip2721"
